Commit message: rearrange launch and urdf files
general:
- components which have an own package have their urdf and launch files
  in the package (kurt_base, kurt_teleop). Composed robots and other
  parts have their urdf in the kurt_description and the launch files in
  the kurt_bringup packages (in accordence with the pr2 setup).

urdf:
- every robot is composed out of a base (indoor, outdoor) and
  different tops (kurt2, kurt360,..)
- tops are again composed out of different parts (sick_lms200,
  rotunit,...)
- generic xacro parameter should go into kurt_description/common.xacro
- complete robot urdfs should go into kurt_description/robots/
- kurt tops are in kurt_description/tops/
- other parts are in kurt_description/parts/

launch:
- typical robot setups can be launch from kurt_bringup/launch/
- launch scripts for packages imported from ros should are in
  kurt_bringup/launch/
- kurt_base: launch files for indoor, outdoor and fast kurt_bases
- kurt_teleop: cyborgevo and keyboard launch files

File: kurt_description/robots/kurtX.urdf.xacro (robot description, xacro)
@@ -2,5 +2,6 @@
 <robot
   xmlns:xacro="http://ros.org/wiki/xacro"
-  name="kurt360">
+  name="kurtX">
+  <include filename="$(find kurt_description)/common.xacro" />
   <include filename="$(find kurt_base)/urdf/kurt_outdoor.urdf.xacro" />
   <include filename="$(find kurt_description)/tops/kurt360.urdf.xacro" />
@@ -13,4 +14,5 @@
     <child link="laser_rot_mount_link" />
     <parent link="kurt360_top" />
+    <origin xyz="0 0 0" rpy="0 0 ${M_PI/2}" />
   </joint>
 </robot>
