Commit message: removed kurt_top link again

File: kurt_description/robots/kurt2_indoor.urdf.xacro (robot description, xacro)
@@ -5,8 +5,3 @@
   <include filename="$(find kurt_base)/urdf/kurt_indoor.urdf.xacro" />
   <include filename="$(find kurt_description)/tops/kurt2.urdf.xacro" />
-  <joint name="top_base_joint" type="fixed">
-    <origin xyz="0 0 0.03" rpy="0 0 0" />
-    <parent link="base_link" />
-    <child link="kurt_top" />
-  </joint>
 </robot>

File: kurt_description/tops/kurt2.urdf.xacro (robot description, xacro)
@@ -3,7 +3,4 @@
   xmlns:xacro="http://ros.org/wiki/xacro">
   <include filename="$(find kurt_description)/parts/sick_lms200.urdf.xacro" />
-  <!-- a virtual link, directly above base_link in the center of the top;
-       this is the root link of the top -->
-  <link name="kurt_top" />
   <link name="laptop_structure">
     <visual>
@@ -26,7 +23,7 @@
   </link>
   <joint name="top_to_structure" type="fixed">
-    <parent link="kurt_top" />
+    <parent link="base_link" />
     <child link="laptop_structure" />
-    <origin xyz="-0.05 0 0" rpy="0 0 0" />
+    <origin xyz="-0.05 0 0.03" rpy="0 0 0" />
   </joint>
   <joint name="structure_to_laser" type="fixed">
