Commit message: reduced distance between top and base

File: kurt_description/robots/kurt360.urdf.xacro (robot description, xacro)
@@ -8,5 +8,5 @@
     <child link="kurt360_top" />
     <parent link="base_link" />
-    <origin xyz="0 0 0.1075" />
+    <origin xyz="0 0 0.07" />
   </joint>
 </robot>

File: kurt_description/robots/kurtX.urdf.xacro (robot description, xacro)
@@ -8,5 +8,5 @@
     <child link="kurtX_top" />
     <parent link="base_link" />
-    <origin xyz="0 0 0.1075" />
+    <origin xyz="0 0 0.07" />
   </joint>
 </robot>

Commit message: final fixes to kurt360 URDF

File: kurt_description/robots/kurt360.urdf.xacro (robot description, xacro)
@@ -3,10 +3,12 @@
   xmlns:xacro="http://ros.org/wiki/xacro"
   name="kurt360">
+  <xacro:property name="top_y_offset" value="0.009" />
+  <xacro:property name="base_z_offset" value="0.03" /> <!-- distance from base_link to top of cover surface -->
   <include filename="$(find kurt_description)/bases/kurt_outdoor.urdf.xacro" />
   <include filename="$(find kurt_description)/tops/kurt360_top.urdf.xacro" />
   <joint name="top_base_joint" type="fixed">
+    <parent link="base_link" />
     <child link="kurt360_top" />
-    <parent link="base_link" />
-    <origin xyz="0 0 0.07" />
+    <origin xyz="0 ${top_y_offset} ${base_z_offset + top_z/2}" />
   </joint>
 </robot>

File: kurt_description/tops/kurt360_top.urdf.xacro (robot description, xacro)
@@ -8,4 +8,5 @@
   <xacro:property name="top_z" value="0.08" />
   <xacro:property name="top_mass" value="2.0" />
+  <xacro:property name="rotunit_box_y_offset" value="-0.01" />
   <link name="kurt360_top">
     <visual>
@@ -28,5 +29,5 @@
     <child link="rotunit_box_link" />
     <parent link="kurt360_top" />
-    <origin xyz="0 0 ${top_z/2 + rotunit_box_z/2}" rpy="0 0 0" />
+    <origin xyz="0 ${rotunit_box_y_offset} ${top_z/2 + rotunit_box_z/2}" rpy="0 0 0" />
   </joint>
 </robot>
