Commit message: fixed laser joint name

File: kurt_description/tops/kurt2.urdf.xacro (robot description, xacro)
@@ -14,5 +14,5 @@
     </visual>
   </link>
-  <joint name="laser_rot_joint" type="fixed">
+  <joint name="laser_joint" type="fixed">
     <parent link="kurt2_top" />
     <child link="laser" />
