Commit message: kurtana: add SICK TiM310 laser

File: kurt_description/tops/kurtana_top.urdf.xacro (robot description, xacro)
@@ -22,4 +22,13 @@
     <origin xyz="${kinect_x_offset} 0 ${kinect_z_offset}" rpy="0 0 0"/>
   </joint>
+  <!-- ************************* -->
+  <!-- *** SICK TiM3xx laser *** -->
+  <!-- ************************* -->
+  <include filename="$(find sick_tim3xx)/urdf/sick_tim3xx.urdf.xacro" />
+  <joint name="kurtana_laser_joint" type="fixed">
+    <parent link="kurtana_baseplate_link" />
+    <child link="laser_mount_link" />
+    <origin xyz="${baseplate_length/2 - sick_tim3xx_length/2} 0 ${baseplate_height/2}" rpy="0 0 0" />
+  </joint>
   <!-- **************************** -->
   <!-- *** Neuronics Katana Arm *** -->
@@ -27,7 +36,7 @@
   <include filename="$(find katana_description)/urdf/katana_450_6m90a_with_controlbox.urdf.xacro" />
   <joint name="kurtana_baseplate_controlbox_joint" type="fixed">
-    <origin xyz="0.05 0 ${baseplate_height*1.5}" rpy="0 0 0" />
     <parent link="kurtana_baseplate_link" />
     <child link="katana_internal_controlbox_link" />
+    <origin xyz="0.05 0 ${baseplate_height*1.5}" rpy="0 0 0" />
   </joint>
 </robot>

Commit message: include kinect_pattern in old kurtana_top

File: kurt_description/tops/kurtana_top.urdf.xacro (robot description, xacro)
@@ -36,4 +36,10 @@
   <!-- **************************** -->
   <include filename="$(find katana_description)/urdf/katana_450_6m90a_with_controlbox.urdf.xacro" />
+  <link name="katana_pattern"></link>
+  <joint name="katana_pattern_joint" type="fixed">
+    <parent link="katana_motor4_lift_link"/>
+    <child  link="katana_pattern" />
+    <origin xyz=".075 -.035 0.00" rpy="1.571 -1.571 0.151"/>
+  </joint>
   <joint name="kurtana_baseplate_controlbox_joint" type="fixed">
     <parent link="kurtana_baseplate_link" />
