Commit message: backup gazebo stuff

File: kurt_gazebo/kurt.urdf.xacro (robot description, xacro)
@@ -1,3 +1,4 @@
 <?xml version="1.0"?>
+<<<<<<< HEAD
 <robot name="kurt" xmlns:xacro="http://ros.org/wiki/xacro">
   <xacro:property name="PI" value="3.14159" />
@@ -10,4 +11,8 @@
       </geometry>
     </collision>
+=======
+<robot name="kurt">
+  <link name="body">
+>>>>>>> backup gazebo stuff
     <inertial>
       <origin xyz="0.0 0.0 0.0" />
@@ -18,4 +23,5 @@
       <origin xyz="0.0 0.0 0.0"/>
       <geometry>
+<<<<<<< HEAD
         <box size="${size}" />
       </geometry>
@@ -90,3 +96,18 @@
     <material>Gazebo/Grey</material>
   </gazebo>
+=======
+        <box size="2.0 1.0 1.0" />
+      </geometry>
+    </visual>
+    <collision>
+      <origin xyz="0.0 0.0 0.0"/>
+      <geometry>
+        <box size="1.0 1.0 1.0" />
+      </geometry>
+    </collision>
+  </link>
+  <gazebo reference="body">
+    <material>Gazebo/Red</material>
+  </gazebo>
+>>>>>>> backup gazebo stuff
 </robot>

Commit message: fixed kurt_gazebo

File: kurt_gazebo/kurt.urdf.xacro (robot description, xacro)
@@ -1,4 +1,3 @@
 <?xml version="1.0"?>
-<<<<<<< HEAD
 <robot name="kurt" xmlns:xacro="http://ros.org/wiki/xacro">
   <xacro:property name="PI" value="3.14159" />
@@ -11,8 +10,4 @@
       </geometry>
     </collision>
-=======
-<robot name="kurt">
-  <link name="body">
->>>>>>> backup gazebo stuff
     <inertial>
       <origin xyz="0.0 0.0 0.0" />
@@ -23,5 +18,4 @@
       <origin xyz="0.0 0.0 0.0"/>
       <geometry>
-<<<<<<< HEAD
         <box size="${size}" />
       </geometry>
@@ -96,18 +90,3 @@
     <material>Gazebo/Grey</material>
   </gazebo>
-=======
-        <box size="2.0 1.0 1.0" />
-      </geometry>
-    </visual>
-    <collision>
-      <origin xyz="0.0 0.0 0.0"/>
-      <geometry>
-        <box size="1.0 1.0 1.0" />
-      </geometry>
-    </collision>
-  </link>
-  <gazebo reference="body">
-    <material>Gazebo/Red</material>
-  </gazebo>
->>>>>>> backup gazebo stuff
 </robot>
