Commit message: added collision models to urdf
- added Harting plug to rotunit (as additional model for now)
- fixed some numbers and names along the way

File: kurt_base/urdf/kurt_outdoor.urdf.xacro (robot description, xacro)
@@ -5,5 +5,5 @@
     <visual>
       <geometry>
-        <box size=".43 .43 .23" />
+        <box size=".43 .325 .215" />
       </geometry>
       <material name="red" >
@@ -11,4 +11,9 @@
       </material>
     </visual>
+    <collision>
+      <geometry>
+        <box size=".43 .325 .215" />
+      </geometry>
+    </collision>
   </link>
 </robot>

File: kurt_base/urdf/rotunit.urdf.xacro (robot description, xacro)
@@ -14,10 +14,35 @@
       </material>
     </visual>
+    <collision>
+      <geometry>
+        <box size=".18 .18 .143" />
+      </geometry>
+    </collision>
   </link>
   <joint name="laser_rot_joint" type="continuous">
     <parent link="laser_rot_mount_link" />
     <child link="laser" />
-    <origin xyz="0 0 0.22" rpy="${-M_PI/2} 0 0" />
+    <origin xyz="0 0 0.143" rpy="${-M_PI/2} 0 0" />
     <axis xyz="0 1 0" />
   </joint>
+  <link name="harting_rot_link">
+    <visual>
+      <geometry>
+        <box size=".1 .13 .06" />
+      </geometry>
+      <material name="silver" >
+        <color rgba="0.2 0.2 0.2 1" />
+      </material>
+    </visual>
+    <collision>
+      <geometry>
+        <box size=".1 .13 .06" />
+      </geometry>
+    </collision>
+  </link>
+  <joint name="harting_rot_joint" type="fixed">
+    <parent link="laser_rot_mount_link" />
+    <child link="harting_rot_link" />
+    <origin xyz="-0.09 0 0" />
+  </joint>
 </robot>

File: kurt_description/parts/sick_lms200.urdf.xacro (robot description, xacro)
@@ -4,11 +4,16 @@
   <link name="laser">
     <visual>
-	    <geometry>
-	      <box size=".156 .155 .185" />
-	    </geometry>
-    	<material name="blue" >
-      		<color rgba="0 0 1 1" />
-    	</material>
-  	</visual>
+      <geometry>
+        <box size=".156 .155 .185" />
+      </geometry>
+      <material name="blue" >
+        <color rgba="0 0 1 1" />
+      </material>
+    </visual>
+    <collision>
+      <geometry>
+        <box size=".156 .155 .185" />
+      </geometry>
+    </collision>
   </link>
 </robot>

File: kurt_description/robots/kurt360.urdf.xacro (robot description, xacro)
@@ -5,12 +5,8 @@
   <include filename="$(find kurt_base)/urdf/kurt_outdoor.urdf.xacro" />
   <include filename="$(find kurt_description)/tops/kurt360.urdf.xacro" />
-  <include filename="$(find kurt_base)/urdf/rotunit.urdf.xacro" />
   <joint name="top_base_joint" type="fixed">
     <child link="kurt360_top" />
     <parent link="base_link" />
-  </joint>
-  <joint name="laser_top_joint" type="fixed">
-    <child link="laser_rot_mount_link" />
-    <parent link="kurt360_top" />
+    <origin xyz="0 0 0.1075" />
   </joint>
 </robot>

File: kurt_description/robots/kurtX.urdf.xacro (robot description, xacro)
@@ -3,16 +3,10 @@
   xmlns:xacro="http://ros.org/wiki/xacro"
   name="kurtX">
-  <include filename="$(find kurt_description)/common.xacro" />
   <include filename="$(find kurt_base)/urdf/kurt_outdoor.urdf.xacro" />
-  <include filename="$(find kurt_description)/tops/kurt360.urdf.xacro" />
-  <include filename="$(find kurt_base)/urdf/rotunit.urdf.xacro" />
+  <include filename="$(find kurt_description)/tops/kurtX.urdf.xacro" />
   <joint name="top_base_joint" type="fixed">
-    <child link="kurt360_top" />
+    <child link="kurtX_top" />
     <parent link="base_link" />
-  </joint>
-  <joint name="laser_top_joint" type="fixed">
-    <child link="laser_rot_mount_link" />
-    <parent link="kurt360_top" />
-    <origin xyz="0 0 0" rpy="0 0 ${M_PI/2}" />
+    <origin xyz="0 0 0.1075" />
   </joint>
 </robot>

File: kurt_description/tops/kurtX.urdf.xacro (robot description, xacro)
@@ -4,5 +4,5 @@
   <include filename="$(find kurt_description)/common.xacro" />
   <include filename="$(find kurt_base)/urdf/rotunit.urdf.xacro" />
-  <link name="kurt360_top">
+  <link name="kurtX_top">
     <visual>
       <geometry>
@@ -22,5 +22,5 @@
   <joint name="laser_top_joint" type="fixed">
     <child link="laser_rot_mount_link" />
-    <parent link="kurt360_top" />
+    <parent link="kurtX_top" />
     <origin xyz="0 0 0.08" rpy="0 0 ${M_PI/2}" />
   </joint>

Commit message: added meshes to kurt_outdoor URDF

File: kurt_base/urdf/kurt_outdoor.urdf.xacro (robot description, xacro)
@@ -1,7 +1,31 @@
 <?xml version="1.0"?>
 <robot
-  xmlns:xacro="http://ros.org/wiki/xacro">
+  xmlns:xacro="http://ros.org/wiki/xacro"
+  name="kurt_outdoor_base">
+  <xacro:property name="PI" value="3.14159" />
+  <!-- TODO: measure all these values on a real KURT -->
+  <xacro:property name="wheel_width" value="0.04" />
+  <xacro:property name="wheel_radius" value="0.08244" />
+  <xacro:property name="axis_length" value="0.28" />
+  <xacro:property name="middle_axis_length" value="0.37" />
+  <xacro:property name="wheel_x_offset" value="0.14" />
+  <xacro:property name="wheel_z_offset" value="-0.09" />
   <link name="base_link">
     <visual>
+      <origin xyz="0 0 0" rpy="0 0 0" />
+      <geometry>
+        <mesh filename="package://kurt_description/meshes/kurt_base_outdoor.stl" />
+      </geometry>
+      <material name="red" >
+        <color rgba="1 0 0 1" />
+      </material>
+    </visual>
+    <collision>
+      <origin xyz="0 0 0" rpy="0 0 0" />
+      <geometry>
+        <mesh filename="package://kurt_description/meshes/kurt_base_outdoor.stl" />
+      </geometry>
+    </collision>
+    <!-- <visual>
       <geometry>
         <box size=".43 .325 .215" />
@@ -10,10 +34,38 @@
         <color rgba="1 0 0 1" />
       </material>
-    </visual>
-    <collision>
+    </visual> -->
+  </link>
+  <xacro:macro name="kurt_wheel" params="name xyz">
+    <link name="kurt_wheel_${name}">
+      <visual>
+        <origin xyz="0 0 0" rpy="0 0 0" />
+        <geometry>
+          <mesh filename="package://kurt_description/meshes/kurt_wheel_outdoor.stl" />
+        </geometry>
+        <material name="blackish"><color rgba="0.1 0.1 0.1 1"/></material>
+      </visual>
+      <collision>
+        <origin xyz="0 0 0" rpy="0 0 0" />
+        <geometry>
+          <mesh filename="package://kurt_description/meshes/kurt_wheel_outdoor.stl" />
+        </geometry>
+        <!--
       <geometry>
-        <box size=".43 .325 .215" />
-      </geometry>
+        <cylinder length="${wheel_width}" radius="${wheel_radius}" />
+      </geometry>-->
     </collision>
   </link>
+  <joint name="body_to_wheel_${name}" type="continuous">
+    <origin xyz="${xyz}" rpy="0 0 0" />
+    <parent link="base_link"/>
+    <child link="kurt_wheel_${name}"/>
+    <axis xyz="0 1 0"/>
+  </joint>
+</xacro:macro>
+<xacro:kurt_wheel name="left_front" xyz="${wheel_x_offset} ${axis_length/2} ${wheel_z_offset}" />
+<xacro:kurt_wheel name="left_middle" xyz="0 ${middle_axis_length/2} ${wheel_z_offset}" />
+<xacro:kurt_wheel name="left_rear" xyz="${-wheel_x_offset} ${axis_length/2} ${wheel_z_offset}" />
+<xacro:kurt_wheel name="right_front" xyz="${wheel_x_offset} ${-axis_length/2} ${wheel_z_offset}" />
+<xacro:kurt_wheel name="right_middle" xyz="0 ${-middle_axis_length/2} ${wheel_z_offset}" />
+<xacro:kurt_wheel name="right_rear" xyz="${-wheel_x_offset} ${-axis_length/2} ${wheel_z_offset}" />
 </robot>

Commit message: added gazebo to kurt outdoor base

File: kurt_base/urdf/kurt_outdoor.urdf.xacro (robot description, xacro)
@@ -1,4 +1,6 @@
 <?xml version="1.0"?>
-<robot
+<robot xmlns:controller="http://playerstage.sourceforge.net/gazebo/xmlschema/#controller"
+  xmlns:interface="http://playerstage.sourceforge.net/gazebo/xmlschema/#interface"
+  xmlns:sensor="http://playerstage.sourceforge.net/gazebo/xmlschema/#sensor"
   xmlns:xacro="http://ros.org/wiki/xacro"
   name="kurt_outdoor_base">
@@ -11,4 +13,5 @@
   <xacro:property name="wheel_x_offset" value="0.14" />
   <xacro:property name="wheel_z_offset" value="-0.10" />
+  <xacro:property name="turning_adaptation" value="0.60" />  <!-- physical kurt outdoor: 0.46 -->
   <link name="base_link">
     <visual>
@@ -43,4 +46,36 @@
     </inertial>
   </link>
+  <gazebo reference="base_link">
+    <material value="Gazebo/Red" />
+  </gazebo>
+  <gazebo>
+    <controller:gazebo_ros_kurt name="kurt_controller" plugin="libgazebo_ros_kurt.so">
+      <alwaysOn>true</alwaysOn>
+      <!-- <node_namespace>kurt_controller</node_namespace> -->
+      <left_front_wheel_joint>body_to_wheel_left_front</left_front_wheel_joint>
+      <left_middle_wheel_joint>body_to_wheel_left_middle</left_middle_wheel_joint>
+      <left_rear_wheel_joint>body_to_wheel_left_rear</left_rear_wheel_joint>
+      <right_front_wheel_joint>body_to_wheel_right_front</right_front_wheel_joint>
+      <right_middle_wheel_joint>body_to_wheel_right_middle</right_middle_wheel_joint>
+      <right_rear_wheel_joint>body_to_wheel_right_rear</right_rear_wheel_joint>
+      <wheel_separation>${middle_axis_length}</wheel_separation>
+      <wheel_diameter>${2*wheel_radius}</wheel_diameter>
+      <turning_adaptation>${turning_adaptation}</turning_adaptation>
+      <torque>2.0</torque>
+      <updateRate>40.0</updateRate>
+    </controller:gazebo_ros_kurt>
+  </gazebo>
+  <!-- publish ground truth for pose of base_footprint -->
+  <gazebo>
+    <controller:gazebo_ros_p3d name="base_footprint_controller" plugin="libgazebo_ros_p3d.so">
+      <alwaysOn>true</alwaysOn>
+      <updateRate>30.0</updateRate>
+      <bodyName>base_footprint</bodyName>
+      <topicName>base_footprint_pose_ground_truth</topicName>
+      <gaussianNoise>0.0</gaussianNoise>
+      <frameName>map</frameName>
+      <interface:position name="base_footprint_p3d_position_iface" />
+    </controller:gazebo_ros_p3d>
+  </gazebo>
   <xacro:macro name="kurt_wheel" params="name xyz">
     <link name="kurt_wheel_${name}">
@@ -73,4 +108,7 @@
       <axis xyz="0 1 0"/>
     </joint>
+    <gazebo reference="kurt_wheel_${name}">
+      <material value="Gazebo/Grey" />
+    </gazebo>
   </xacro:macro>
   <xacro:kurt_wheel name="left_front" xyz="${wheel_x_offset} ${axis_length/2} ${wheel_z_offset}" />
@@ -82,5 +120,14 @@
   <!-- base_footprint is a fictitious link(frame) that is on the ground right below base_link origin,
        navigation stack dedpends on this frame -->
-  <link name="base_footprint" />
+  <link name="base_footprint">
+    <!-- this needs to have a fake inertial element, otherwise all children will be ignored by Gazebo -->
+    <inertial>
+      <mass value="0.0001" />
+      <origin xyz="0 0 0" />
+      <inertia ixx="0.0001" ixy="0.0" ixz="0.0"
+        iyy="0.0001" iyz="0.0"
+        izz="0.0001" />
+    </inertial>
+  </link>
   <joint name="base_footprint_joint" type="fixed">
     <origin xyz="0 0 ${-wheel_z_offset + wheel_radius}" rpy="0 0 0" />
