Commit message: added inertial values to kurt

File: kurt_base/urdf/kurt_indoor.urdf.xacro (robot description, xacro)
@@ -35,4 +35,11 @@
       </material>
     </visual> -->
+    <inertial>
+      <mass value="7.0" />
+      <origin xyz="0.0 0.0 -0.040426445" />
+      <inertia ixx="0.053184933" ixy="0.0" ixz="0.0"
+        iyy="0.086499893" iyz="0.0"
+        izz="0.107785706" />
+    </inertial>
   </link>
   <xacro:macro name="kurt_wheel" params="name xyz rotate_visual">
@@ -56,4 +63,11 @@
       </geometry>-->
     </collision>
+    <inertial>
+      <mass value="0.075" />
+      <origin xyz="0 0 0" />
+      <inertia ixx="0.000066031" ixy="0.0" ixz="0.0"
+        iyy="0.000129786" iyz="0.0"
+        izz="0.000066031" />
+    </inertial>
   </link>
   <joint name="body_to_wheel_${name}" type="continuous">

File: kurt_base/urdf/kurt_outdoor.urdf.xacro (robot description, xacro)
@@ -35,4 +35,11 @@
       </material>
     </visual> -->
+    <inertial>
+      <mass value="7.0" />
+      <origin xyz="0.0 0.0 -0.040426445" />
+      <inertia ixx="0.053184933" ixy="0.0" ixz="0.0"
+        iyy="0.086499893" iyz="0.0"
+        izz="0.107785706" />
+    </inertial>
   </link>
   <xacro:macro name="kurt_wheel" params="name xyz">
@@ -55,4 +62,11 @@
       </geometry>-->
     </collision>
+    <inertial>
+      <mass value="0.15" />
+      <origin xyz="0 0 0" />
+      <inertia ixx="0.000177810" ixy="0.0" ixz="0.0"
+        iyy="0.000332643" iyz="0.0"
+        izz="0.000177810" />
+    </inertial>
   </link>
   <joint name="body_to_wheel_${name}" type="continuous">

File: kurt_base/urdf/rotunit.urdf.xacro (robot description, xacro)
@@ -5,8 +5,16 @@
   <include filename="$(find kurt_description)/common.xacro" />
   <include filename="$(find kurt_description)/parts/sick_lms200.urdf.xacro" />
+  <xacro:property name="laser_rot_mount_x" value="0.18" />
+  <xacro:property name="laser_rot_mount_y" value="0.18" />
+  <xacro:property name="laser_rot_mount_z" value="0.143" />
+  <xacro:property name="laser_rot_mount_mass" value="1.5" />
+  <xacro:property name="harting_rot_x" value="0.05" />
+  <xacro:property name="harting_rot_y" value="0.13" />
+  <xacro:property name="harting_rot_z" value="0.06" />
+  <xacro:property name="harting_rot_mass" value="0.2" />
   <link name="laser_rot_mount_link">
     <visual>
       <geometry>
-        <box size=".18 .18 .143" />
+        <box size="${laser_rot_mount_x} ${laser_rot_mount_y} ${laser_rot_mount_z}" />
       </geometry>
       <material name="silver" >
@@ -16,12 +24,13 @@
     <collision>
       <geometry>
-        <box size=".18 .18 .143" />
+        <box size="${laser_rot_mount_x} ${laser_rot_mount_y} ${laser_rot_mount_z}" />
       </geometry>
     </collision>
+    <xacro:box_inertial x="${laser_rot_mount_x}" y="${laser_rot_mount_y}" z="${laser_rot_mount_z}" mass="${laser_rot_mount_mass}" />
   </link>
   <joint name="laser_rot_joint" type="continuous">
     <parent link="laser_rot_mount_link" />
     <child link="laser" />
-    <origin xyz="0 0 0.143" rpy="${-M_PI/2} 0 0" />
+    <origin xyz="0 0 ${laser_rot_mount_z}" rpy="${-M_PI/2} 0 0" />
     <axis xyz="0 1 0" />
   </joint>
@@ -29,20 +38,19 @@
     <visual>
       <geometry>
-        <box size=".1 .13 .06" />
+        <box size="${harting_rot_x} ${harting_rot_y} ${harting_rot_z}" />
       </geometry>
-      <material name="silver" >
-        <color rgba="0.2 0.2 0.2 1" />
-      </material>
+      <material name="silver" />
     </visual>
     <collision>
       <geometry>
-        <box size=".1 .13 .06" />
+        <box size="${harting_rot_x} ${harting_rot_y} ${harting_rot_z}" />
       </geometry>
     </collision>
+    <xacro:box_inertial x="${harting_rot_x}" y="${harting_rot_y}" z="${harting_rot_z}" mass="${harting_rot_mass}" />
   </link>
   <joint name="harting_rot_joint" type="fixed">
     <parent link="laser_rot_mount_link" />
     <child link="harting_rot_link" />
-    <origin xyz="-0.09 0 0" />
+    <origin xyz="${-laser_rot_mount_x/2 - harting_rot_x/2} 0 0" />
   </joint>
 </robot>

File: kurt_description/common.xacro (robot description, xacro)
@@ -1,4 +1,33 @@
 <?xml version="1.0"?>
-<robot>
+<robot
+  xmlns:xacro="http://ros.org/wiki/xacro">
   <property name="M_PI" value="3.1415926535897931" />
+  <!-- see https://secure.wikimedia.org/wikipedia/en/wiki/List_of_moment_of_inertia_tensors -->
+  <xacro:macro name="sphere_inertial" params="radius mass">
+    <inertial>
+      <mass value="${mass}" />
+      <origin xyz="0 0 0" />
+      <inertia ixx="${0.4 * mass * radius * radius}" ixy="0.0" ixz="0.0"
+        iyy="${0.4 * mass * radius * radius}" iyz="0.0"
+        izz="${0.4 * mass * radius * radius}" />
+    </inertial>
+  </xacro:macro>
+  <xacro:macro name="cylinder_inertial" params="radius length mass">
+    <inertial>
+      <mass value="${mass}" />
+      <origin xyz="0 0 0" />
+      <inertia ixx="${0.0833333 * mass * (3 * radius * radius + length * length)}" ixy="0.0" ixz="0.0"
+        iyy="${0.0833333 * mass * (3 * radius * radius + length * length)}" iyz="0.0"
+        izz="${0.5 * mass * radius * radius}" />
+    </inertial>
+  </xacro:macro>
+  <xacro:macro name="box_inertial" params="x y z mass">
+    <inertial>
+      <mass value="${mass}" />
+      <origin xyz="0 0 0" />
+      <inertia ixx="${0.0833333 * mass * (y*y + z*z)}" ixy="0.0" ixz="0.0"
+        iyy="${0.0833333 * mass * (x*x + z*z)}" iyz="0.0"
+        izz="${0.0833333 * mass * (x*x + y*y)}" />
+    </inertial>
+  </xacro:macro>
 </robot>

File: kurt_description/parts/sick_lms200.urdf.xacro (robot description, xacro)
@@ -17,4 +17,11 @@
       </geometry>
     </collision>
+    <inertial>
+      <mass value="2.0" />
+      <origin xyz="-0.022849644 0.000005772 0.040232937" />
+      <inertia ixx="0.009318238" ixy="-0.000000024" ixz="-0.000148360"
+        iyy="0.009251799" iyz="0.000000400"
+        izz="0.007478235" />
+    </inertial>
   </link>
   <gazebo reference="laser">

File: kurt_description/parts/sick_s300.urdf.xacro (robot description, xacro)
@@ -2,13 +2,19 @@
 <robot
   xmlns:xacro="http://ros.org/wiki/xacro">
+  <include filename="$(find kurt_description)/common.xacro" />
+  <xacro:property name="laser_x" value="0.156" />
+  <xacro:property name="laser_y" value="0.155" />
+  <xacro:property name="laser_z" value="0.185" />
+  <xacro:property name="laser_mass" value="2.0" />
   <link name="laser">
     <visual>
 	    <geometry>
-	      <box size=".156 .155 .185" />
+        <box size="${laser_x} ${laser_y} ${laser_z}" />
 	    </geometry>
     	<material name="blue" >
       		<color rgba="0 0 1 1" />
     	</material>
-  	</visual>
+    </visual>
+    <xacro:box_inertial x="${laser_x}" y="${laser_y}" z="${laser_z}" mass="${laser_mass}" />
   </link>
 </robot>

File: kurt_description/tops/kurt2.urdf.xacro (robot description, xacro)
@@ -12,4 +12,16 @@
       </geometry>
     </visual>
+    <collision>
+      <geometry>
+        <mesh filename="package://kurt_description/meshes/laptop_structure.dae" />
+      </geometry>
+    </collision>
+    <inertial>
+      <mass value="2.0" />
+      <origin xyz="-0.005401183 0.0 0.141356018" />
+      <inertia ixx="0.022277280" ixy="-0.000000004" ixz="-0.001009999"
+        iyy="0.017783837" iyz="0.0"
+        izz="0.025523417" />
+    </inertial>
   </link>
   <joint name="top_to_structure" type="fixed">

File: kurt_description/tops/kurt360.urdf.xacro (robot description, xacro)
@@ -4,8 +4,12 @@
   <include filename="$(find kurt_description)/common.xacro" />
   <include filename="$(find kurt_base)/urdf/rotunit.urdf.xacro" />
+  <xacro:property name="top_x" value="0.36" />
+  <xacro:property name="top_y" value="0.28" />
+  <xacro:property name="top_z" value="0.08" />
+  <xacro:property name="top_mass" value="2.0" />
   <link name="kurt360_top">
     <visual>
       <geometry>
-        <box size=".36 .28 .08" />
+        <box size="${top_x} ${top_y} ${top_z}" />
       </geometry>
       <origin xyz="0 0 0" rpy="0 0 0" />
@@ -16,12 +20,13 @@
     <collision>
       <geometry>
-        <box size=".36 .28 .08" />
+        <box size="${top_x} ${top_y} ${top_z}" />
       </geometry>
     </collision>
+    <xacro:box_inertial x="${top_x}" y="${top_y}" z="${top_z}" mass="${top_mass}" />
   </link>
   <joint name="laser_top_joint" type="fixed">
     <child link="laser_rot_mount_link" />
     <parent link="kurt360_top" />
-    <origin xyz="0 0 0.08" rpy="0 0 ${M_PI/2}" />
+    <origin xyz="0 0 ${top_z}" rpy="0 0 ${M_PI/2}" />
   </joint>
 </robot>

File: kurt_description/tops/kurtX.urdf.xacro (robot description, xacro)
@@ -4,8 +4,12 @@
   <include filename="$(find kurt_description)/common.xacro" />
   <include filename="$(find kurt_base)/urdf/rotunit.urdf.xacro" />
+  <xacro:property name="top_x" value="0.36" />
+  <xacro:property name="top_y" value="0.28" />
+  <xacro:property name="top_z" value="0.08" />
+  <xacro:property name="top_mass" value="2.0" />
   <link name="kurtX_top">
     <visual>
       <geometry>
-        <box size=".36 .28 .08" />
+        <box size="${top_x} ${top_y} ${top_z}" />
       </geometry>
       <origin xyz="0 0 0" rpy="0 0 0" />
@@ -16,12 +20,13 @@
     <collision>
       <geometry>
-        <box size=".36 .28 .08" />
+        <box size="${top_x} ${top_y} ${top_z}" />
       </geometry>
     </collision>
+    <xacro:box_inertial x="${top_x}" y="${top_y}" z="${top_z}" mass="${top_mass}" />
   </link>
   <joint name="laser_top_joint" type="fixed">
     <child link="laser_rot_mount_link" />
     <parent link="kurtX_top" />
-    <origin xyz="0 0 0.08" rpy="0 0 ${M_PI/2}" />
+    <origin xyz="0 0 ${top_z}" rpy="0 0 ${M_PI/2}" />
   </joint>
 </robot>

Commit message: fixed wheel scale

File: kurt_base/urdf/kurt_indoor.urdf.xacro (robot description, xacro)
@@ -7,8 +7,8 @@
   <xacro:property name="wheel_width" value="0.02" />
   <xacro:property name="wheel_radius" value="0.060319723" />
-  <xacro:property name="axis_length" value="0.25" />
-  <xacro:property name="middle_axis_length" value="0.25" />
-  <xacro:property name="wheel_x_offset" value="0.12" />
-  <xacro:property name="wheel_z_offset" value="-0.12" />
+  <xacro:property name="axis_length" value="0.26" />
+  <xacro:property name="middle_axis_length" value="0.26" />
+  <xacro:property name="wheel_x_offset" value="0.13" />
+  <xacro:property name="wheel_z_offset" value="-0.10" />
   <link name="base_link">
     <visual>

File: kurt_base/urdf/kurt_outdoor.urdf.xacro (robot description, xacro)
@@ -10,5 +10,5 @@
   <xacro:property name="middle_axis_length" value="0.37" />
   <xacro:property name="wheel_x_offset" value="0.14" />
-  <xacro:property name="wheel_z_offset" value="-0.09" />
+  <xacro:property name="wheel_z_offset" value="-0.10" />
   <link name="base_link">
     <visual>

File: kurt_base/urdf/rotunit.urdf.xacro (robot description, xacro)
@@ -32,5 +32,5 @@
     <parent link="laser_rot_mount_link" />
     <child link="laser" />
-    <origin xyz="0 0 ${laser_rot_mount_z}" rpy="${-M_PI/2} 0 0" />
+    <origin xyz="0 0 ${laser_rot_mount_z + 0.005}" rpy="${-M_PI/2} 0 0" />
     <axis xyz="0 1 0" />
   </joint>

Commit message: added base_footprint to urdf

File: kurt_base/urdf/kurt_indoor.urdf.xacro (robot description, xacro)
@@ -57,30 +57,35 @@
         <geometry>
           <mesh filename="package://kurt_description/meshes/kurt_wheel_indoor.dae" />
+          <!-- <cylinder length="${wheel_width}" radius="${wheel_radius}" /> -->
         </geometry>
-        <!--
-      <geometry>
-        <cylinder length="${wheel_width}" radius="${wheel_radius}" />
-      </geometry>-->
-    </collision>
-    <inertial>
-      <mass value="0.075" />
-      <origin xyz="0 0 0" />
-      <inertia ixx="0.000066031" ixy="0.0" ixz="0.0"
-        iyy="0.000129786" iyz="0.0"
-        izz="0.000066031" />
-    </inertial>
-  </link>
-  <joint name="body_to_wheel_${name}" type="continuous">
-    <origin xyz="${xyz}" rpy="0 0 0" />
-    <parent link="base_link"/>
-    <child link="kurt_wheel_${name}"/>
-    <axis xyz="0 1 0"/>
+      </collision>
+      <inertial>
+        <mass value="0.075" />
+        <origin xyz="0 0 0" />
+        <inertia ixx="0.000066031" ixy="0.0" ixz="0.0"
+          iyy="0.000129786" iyz="0.0"
+          izz="0.000066031" />
+      </inertial>
+    </link>
+    <joint name="body_to_wheel_${name}" type="continuous">
+      <origin xyz="${xyz}" rpy="0 0 0" />
+      <parent link="base_link"/>
+      <child link="kurt_wheel_${name}"/>
+      <axis xyz="0 1 0"/>
+    </joint>
+  </xacro:macro>
+  <xacro:kurt_wheel name="left_front" xyz="${wheel_x_offset} ${axis_length/2} ${wheel_z_offset}" rotate_visual="1" />
+  <xacro:kurt_wheel name="left_middle" xyz="0 ${middle_axis_length/2} ${wheel_z_offset}" rotate_visual="1" />
+  <xacro:kurt_wheel name="left_rear" xyz="${-wheel_x_offset} ${axis_length/2} ${wheel_z_offset}" rotate_visual="1" />
+  <xacro:kurt_wheel name="right_front" xyz="${wheel_x_offset} ${-axis_length/2} ${wheel_z_offset}" rotate_visual="0" />
+  <xacro:kurt_wheel name="right_middle" xyz="0 ${-middle_axis_length/2} ${wheel_z_offset}" rotate_visual="0" />
+  <xacro:kurt_wheel name="right_rear" xyz="${-wheel_x_offset} ${-axis_length/2} ${wheel_z_offset}" rotate_visual="0" />
+  <!-- base_footprint is a fictitious link(frame) that is on the ground right below base_link origin,
+       navigation stack dedpends on this frame -->
+  <link name="base_footprint" />
+  <joint name="base_footprint_joint" type="fixed">
+    <origin xyz="0 0 ${-wheel_z_offset + wheel_radius}" rpy="0 0 0" />
+    <parent link="base_footprint"/>
+    <child link="base_link" />
   </joint>
-</xacro:macro>
-<xacro:kurt_wheel name="left_front" xyz="${wheel_x_offset} ${axis_length/2} ${wheel_z_offset}" rotate_visual="1" />
-<xacro:kurt_wheel name="left_middle" xyz="0 ${middle_axis_length/2} ${wheel_z_offset}" rotate_visual="1" />
-<xacro:kurt_wheel name="left_rear" xyz="${-wheel_x_offset} ${axis_length/2} ${wheel_z_offset}" rotate_visual="1" />
-<xacro:kurt_wheel name="right_front" xyz="${wheel_x_offset} ${-axis_length/2} ${wheel_z_offset}" rotate_visual="0" />
-<xacro:kurt_wheel name="right_middle" xyz="0 ${-middle_axis_length/2} ${wheel_z_offset}" rotate_visual="0" />
-<xacro:kurt_wheel name="right_rear" xyz="${-wheel_x_offset} ${-axis_length/2} ${wheel_z_offset}" rotate_visual="0" />
 </robot>

File: kurt_base/urdf/kurt_outdoor.urdf.xacro (robot description, xacro)
@@ -56,30 +56,35 @@
         <geometry>
           <mesh filename="package://kurt_description/meshes/kurt_wheel_outdoor.stl" />
+          <!-- <cylinder length="${wheel_width}" radius="${wheel_radius}" /> -->
         </geometry>
-        <!--
-      <geometry>
-        <cylinder length="${wheel_width}" radius="${wheel_radius}" />
-      </geometry>-->
-    </collision>
-    <inertial>
-      <mass value="0.15" />
-      <origin xyz="0 0 0" />
-      <inertia ixx="0.000177810" ixy="0.0" ixz="0.0"
-        iyy="0.000332643" iyz="0.0"
-        izz="0.000177810" />
-    </inertial>
-  </link>
-  <joint name="body_to_wheel_${name}" type="continuous">
-    <origin xyz="${xyz}" rpy="0 0 0" />
-    <parent link="base_link"/>
-    <child link="kurt_wheel_${name}"/>
-    <axis xyz="0 1 0"/>
+      </collision>
+      <inertial>
+        <mass value="0.15" />
+        <origin xyz="0 0 0" />
+        <inertia ixx="0.000177810" ixy="0.0" ixz="0.0"
+          iyy="0.000332643" iyz="0.0"
+          izz="0.000177810" />
+      </inertial>
+    </link>
+    <joint name="body_to_wheel_${name}" type="continuous">
+      <origin xyz="${xyz}" rpy="0 0 0" />
+      <parent link="base_link"/>
+      <child link="kurt_wheel_${name}"/>
+      <axis xyz="0 1 0"/>
+    </joint>
+  </xacro:macro>
+  <xacro:kurt_wheel name="left_front" xyz="${wheel_x_offset} ${axis_length/2} ${wheel_z_offset}" />
+  <xacro:kurt_wheel name="left_middle" xyz="0 ${middle_axis_length/2} ${wheel_z_offset}" />
+  <xacro:kurt_wheel name="left_rear" xyz="${-wheel_x_offset} ${axis_length/2} ${wheel_z_offset}" />
+  <xacro:kurt_wheel name="right_front" xyz="${wheel_x_offset} ${-axis_length/2} ${wheel_z_offset}" />
+  <xacro:kurt_wheel name="right_middle" xyz="0 ${-middle_axis_length/2} ${wheel_z_offset}" />
+  <xacro:kurt_wheel name="right_rear" xyz="${-wheel_x_offset} ${-axis_length/2} ${wheel_z_offset}" />
+  <!-- base_footprint is a fictitious link(frame) that is on the ground right below base_link origin,
+       navigation stack dedpends on this frame -->
+  <link name="base_footprint" />
+  <joint name="base_footprint_joint" type="fixed">
+    <origin xyz="0 0 ${-wheel_z_offset + wheel_radius}" rpy="0 0 0" />
+    <parent link="base_footprint"/>
+    <child link="base_link" />
   </joint>
-</xacro:macro>
-<xacro:kurt_wheel name="left_front" xyz="${wheel_x_offset} ${axis_length/2} ${wheel_z_offset}" />
-<xacro:kurt_wheel name="left_middle" xyz="0 ${middle_axis_length/2} ${wheel_z_offset}" />
-<xacro:kurt_wheel name="left_rear" xyz="${-wheel_x_offset} ${axis_length/2} ${wheel_z_offset}" />
-<xacro:kurt_wheel name="right_front" xyz="${wheel_x_offset} ${-axis_length/2} ${wheel_z_offset}" />
-<xacro:kurt_wheel name="right_middle" xyz="0 ${-middle_axis_length/2} ${wheel_z_offset}" />
-<xacro:kurt_wheel name="right_rear" xyz="${-wheel_x_offset} ${-axis_length/2} ${wheel_z_offset}" />
 </robot>

Commit message: added gazebo elements to kurt_indoor urdf

File: kurt_base/urdf/kurt_indoor.urdf.xacro (robot description, xacro)
@@ -1,4 +1,6 @@
 <?xml version="1.0"?>
-<robot
+<robot xmlns:controller="http://playerstage.sourceforge.net/gazebo/xmlschema/#controller"
+  xmlns:interface="http://playerstage.sourceforge.net/gazebo/xmlschema/#interface"
+  xmlns:sensor="http://playerstage.sourceforge.net/gazebo/xmlschema/#sensor"
   xmlns:xacro="http://ros.org/wiki/xacro"
   name="kurt_outdoor_base">
@@ -43,4 +45,23 @@
     </inertial>
   </link>
+  <gazebo reference="base_link">
+    <material value="Gazebo/Black" />
+  </gazebo>
+  <gazebo>
+    <controller:gazebo_ros_kurt name="kurt_controller" plugin="libgazebo_ros_kurt.so">
+      <alwaysOn>true</alwaysOn>
+      <!-- <node_namespace>kurt_controller</node_namespace> -->
+      <left_front_wheel_joint>body_to_wheel_left_front</left_front_wheel_joint>
+      <left_middle_wheel_joint>body_to_wheel_left_middle</left_middle_wheel_joint>
+      <left_rear_wheel_joint>body_to_wheel_left_rear</left_rear_wheel_joint>
+      <right_front_wheel_joint>body_to_wheel_right_front</right_front_wheel_joint>
+      <right_middle_wheel_joint>body_to_wheel_right_middle</right_middle_wheel_joint>
+      <right_rear_wheel_joint>body_to_wheel_right_rear</right_rear_wheel_joint>
+      <wheel_separation>${middle_axis_length}</wheel_separation>
+      <wheel_diameter>${2*wheel_radius}</wheel_diameter>
+      <torque>2.0</torque>
+      <updateRate>1000.0</updateRate>
+    </controller:gazebo_ros_kurt>
+  </gazebo>
   <xacro:macro name="kurt_wheel" params="name xyz rotate_visual">
     <!-- rotate_visual: 0 for right side, 1 for left side -->
@@ -83,5 +104,14 @@
   <!-- base_footprint is a fictitious link(frame) that is on the ground right below base_link origin,
        navigation stack dedpends on this frame -->
-  <link name="base_footprint" />
+  <link name="base_footprint">
+    <!-- this needs to have a fake inertial element, otherwise all children will be ignored by Gazebo -->
+    <inertial>
+      <mass value="0.0001" />
+      <origin xyz="0 0 0" />
+      <inertia ixx="0.0001" ixy="0.0" ixz="0.0"
+        iyy="0.0001" iyz="0.0"
+        izz="0.0001" />
+    </inertial>
+  </link>
   <joint name="base_footprint_joint" type="fixed">
     <origin xyz="0 0 ${-wheel_z_offset + wheel_radius}" rpy="0 0 0" />

Commit message: renamed body_to_wheel_* to *_wheel_joint

File: kurt_base/urdf/kurt_indoor.urdf.xacro (robot description, xacro)
@@ -53,10 +53,10 @@
       <alwaysOn>true</alwaysOn>
       <!-- <node_namespace>kurt_controller</node_namespace> -->
-      <left_front_wheel_joint>body_to_wheel_left_front</left_front_wheel_joint>
-      <left_middle_wheel_joint>body_to_wheel_left_middle</left_middle_wheel_joint>
-      <left_rear_wheel_joint>body_to_wheel_left_rear</left_rear_wheel_joint>
-      <right_front_wheel_joint>body_to_wheel_right_front</right_front_wheel_joint>
-      <right_middle_wheel_joint>body_to_wheel_right_middle</right_middle_wheel_joint>
-      <right_rear_wheel_joint>body_to_wheel_right_rear</right_rear_wheel_joint>
+      <left_front_wheel_joint>left_front_wheel_joint</left_front_wheel_joint>
+      <left_middle_wheel_joint>left_middle_wheel_joint</left_middle_wheel_joint>
+      <left_rear_wheel_joint>left_rear_wheel_joint</left_rear_wheel_joint>
+      <right_front_wheel_joint>right_front_wheel_joint</right_front_wheel_joint>
+      <right_middle_wheel_joint>right_middle_wheel_joint</right_middle_wheel_joint>
+      <right_rear_wheel_joint>right_rear_wheel_joint</right_rear_wheel_joint>
       <wheel_separation>${middle_axis_length}</wheel_separation>
       <wheel_diameter>${2*wheel_radius}</wheel_diameter>
@@ -103,5 +103,5 @@
       </inertial>
     </link>
-    <joint name="body_to_wheel_${name}" type="continuous">
+    <joint name="${name}_wheel_joint" type="continuous">
       <origin xyz="${xyz}" rpy="0 0 0" />
       <parent link="base_link"/>

File: kurt_base/urdf/kurt_outdoor.urdf.xacro (robot description, xacro)
@@ -53,10 +53,10 @@
       <alwaysOn>true</alwaysOn>
       <!-- <node_namespace>kurt_controller</node_namespace> -->
-      <left_front_wheel_joint>body_to_wheel_left_front</left_front_wheel_joint>
-      <left_middle_wheel_joint>body_to_wheel_left_middle</left_middle_wheel_joint>
-      <left_rear_wheel_joint>body_to_wheel_left_rear</left_rear_wheel_joint>
-      <right_front_wheel_joint>body_to_wheel_right_front</right_front_wheel_joint>
-      <right_middle_wheel_joint>body_to_wheel_right_middle</right_middle_wheel_joint>
-      <right_rear_wheel_joint>body_to_wheel_right_rear</right_rear_wheel_joint>
+      <left_front_wheel_joint>left_front_wheel_joint</left_front_wheel_joint>
+      <left_middle_wheel_joint>left_middle_wheel_joint</left_middle_wheel_joint>
+      <left_rear_wheel_joint>left_rear_wheel_joint</left_rear_wheel_joint>
+      <right_front_wheel_joint>right_front_wheel_joint</right_front_wheel_joint>
+      <right_middle_wheel_joint>right_middle_wheel_joint</right_middle_wheel_joint>
+      <right_rear_wheel_joint>right_rear_wheel_joint</right_rear_wheel_joint>
       <wheel_separation>${middle_axis_length}</wheel_separation>
       <wheel_diameter>${2*wheel_radius}</wheel_diameter>
@@ -102,5 +102,5 @@
       </inertial>
     </link>
-    <joint name="body_to_wheel_${name}" type="continuous">
+    <joint name="${name}_wheel_joint" type="continuous">
       <origin xyz="${xyz}" rpy="0 0 0" />
       <parent link="base_link"/>
