Commit message: added sick lms200 mesh

File: kurt_description/parts/sick_lms200.urdf.xacro (robot description, xacro)
@@ -5,5 +5,5 @@
     <visual>
       <geometry>
-        <box size=".156 .155 .185" />
+        <mesh filename="package://kurt_description/meshes/sick_lms-200.stl" />
       </geometry>
       <material name="blue" >
@@ -13,7 +13,11 @@
     <collision>
       <geometry>
-        <box size=".156 .155 .185" />
+        <mesh filename="package://kurt_description/meshes/sick_lms-200.stl" />
+        <!-- <box size=".156 .155 .185" />-->
       </geometry>
     </collision>
   </link>
+  <gazebo reference="laser">
+    <material value="Gazebo/Blue" />
+  </gazebo>
 </robot>

Commit message: added gazebo controller to sick_lms200

File: kurt_description/parts/sick_lms200.urdf.xacro (robot description, xacro)
@@ -1,4 +1,6 @@
 <?xml version="1.0"?>
-<robot
+<robot xmlns:controller="http://playerstage.sourceforge.net/gazebo/xmlschema/#controller"
+  xmlns:interface="http://playerstage.sourceforge.net/gazebo/xmlschema/#interface"
+  xmlns:sensor="http://playerstage.sourceforge.net/gazebo/xmlschema/#sensor"
   xmlns:xacro="http://ros.org/wiki/xacro">
   <link name="laser">
@@ -27,4 +29,25 @@
   <gazebo reference="laser">
     <material value="Gazebo/Blue" />
+    <sensor:ray name="laser">
+      <rayCount>180</rayCount>
+      <rangeCount>180</rangeCount>
+      <laserCount>1</laserCount>
+      <origin>0.0 0.0 0.0</origin>
+      <displayRays>false</displayRays>
+      <minAngle>-90</minAngle>
+      <maxAngle>90</maxAngle>
+      <minRange>0.08</minRange>
+      <maxRange>10.0</maxRange>
+      <resRange>0.01</resRange>
+      <updateRate>75.0</updateRate>
+      <controller:gazebo_ros_laser name="gazebo_ros_laser_controller" plugin="libgazebo_ros_laser.so">
+        <gaussianNoise>0.005</gaussianNoise>
+        <alwaysOn>true</alwaysOn>
+        <updateRate>75.0</updateRate>
+        <topicName>scan</topicName>
+        <frameName>laser</frameName>
+        <interface:laser name="gazebo_ros_laser_iface" />
+      </controller:gazebo_ros_laser>
+    </sensor:ray>
   </gazebo>
 </robot>
