Commit message: add synonyms for openni driver to kinect urdf

File: kurt_description/parts/kinect.urdf.xacro (robot description, xacro)
@@ -68,3 +68,59 @@
     </inertial>
   </link>
+  <!-- ========== synonyms for openni driver ========== -->
+  <joint name="camera_link_joint" type="fixed">
+    <origin xyz="0 0 0" />
+    <parent link="kinect_link" />
+    <child link="camera_link" />
+  </joint>
+  <link name="camera_link">
+    <inertial>
+      <mass value="0.00001" />
+      <origin xyz="0 0 0" />
+      <inertia ixx="1.0" ixy="0.0" ixz="0.0"
+        iyy="1.0" iyz="0.0"
+        izz="1.0" />
+    </inertial>
+  </link>
+  <joint name="camera_depth_joint" type="fixed">
+    <origin xyz="0 0.018 0" rpy="0 0 0" />
+    <parent link="camera_link" />
+    <child link="camera_depth_origin" />
+  </joint>
+  <link name="camera_depth_origin">
+    <inertial>
+      <mass value="0.000001" />
+      <origin xyz="0 0 0" />
+      <inertia ixx="0.0001" ixy="0.0" ixz="0.0"
+        iyy="0.0001" iyz="0.0"
+        izz="0.0001" />
+    </inertial>
+  </link>
+  <joint name="camera_depth_optical_joint" type="fixed">
+    <origin xyz="0 0 0" rpy="${-M_PI/2} 0 ${-M_PI/2}" />
+    <parent link="camera_depth_origin" />
+    <child link="camera_depth" />
+  </joint>
+  <link name="camera_depth">
+    <inertial>
+      <mass value="0.000001" />
+      <origin xyz="0 0 0" />
+      <inertia ixx="0.0001" ixy="0.0" ixz="0.0"
+        iyy="0.0001" iyz="0.0" izz="0.0001" />
+    </inertial>
+  </link>
+  <joint name="camera_rgb_joint" type="fixed">
+    <origin xyz="0 -0.005 0" rpy="0 0 0" />
+    <parent link="camera_link" />
+    <child link="camera_rgb" />
+  </joint>
+  <link name="camera_rgb">
+    <inertial>
+      <mass value="0.000001" />
+      <origin xyz="0 0 0" />
+      <inertia ixx="0.0001" ixy="0.0" ixz="0.0"
+        iyy="0.0001" iyz="0.0"
+        izz="0.0001" />
+    </inertial>
+  </link>
 </robot>

Commit message: fix kinect collision box

File: kurt_description/parts/kinect.urdf.xacro (robot description, xacro)
@@ -15,5 +15,5 @@
     </inertial>
     <visual>
-      <origin xyz=" 0 0 0 " rpy="0 0 0" />
+      <origin xyz="0 0 0" rpy="0 0 0" />
       <geometry>
         <mesh filename="package://kurt_description/meshes/kinect/kinect.dae"/>
@@ -21,5 +21,5 @@
     </visual>
     <collision>
-      <origin xyz="0.0 0.0 0.0" rpy="0 0 0" />
+      <origin xyz="-0.0315 0 -0.017" rpy="0 0 0" />
       <geometry>
         <box size="0.0730 .2760 0.0720"/>

Commit message: removed  duplicate elements in kinect URDF
were added to use with openni driver; instead, set launch file arg
"camera" to "kinect" in openni launch files

File: kurt_description/parts/kinect.urdf.xacro (robot description, xacro)
@@ -4,123 +4,69 @@
   xmlns:interface="http://playerstage.sourceforge.net/gazebo/xmlschema/#interface"
   xmlns:xacro="http://ros.org/wiki/xacro"
-  name="kinect">
+  name="${camera}">
   <property name="M_PI" value="3.1415926535897931" />
-  <link name="kinect_link">
-    <inertial>
-      <mass value="0.00001" />
-      <origin xyz="0 0 0" />
-      <inertia ixx="1.0" ixy="0.0" ixz="0.0"
-        iyy="1.0" iyz="0.0"
-        izz="1.0" />
-    </inertial>
-    <visual>
-      <origin xyz="0 0 0" rpy="0 0 0" />
-      <geometry>
-        <mesh filename="package://kurt_description/meshes/kinect/kinect.dae"/>
-      </geometry>
-    </visual>
-    <collision>
-      <origin xyz="-0.0315 0 -0.017" rpy="0 0 0" />
-      <geometry>
-        <box size="0.0730 .2760 0.0720"/>
-      </geometry>
-    </collision>
-  </link>
-  <joint name="kinect_depth_joint" type="fixed">
-    <origin xyz="0 0.018 0" rpy="0 0 0" />
-    <parent link="kinect_link" />
-    <child link="kinect_depth_origin" />
-  </joint>
-  <link name="kinect_depth_origin">
-    <inertial>
-      <mass value="0.000001" />
-      <origin xyz="0 0 0" />
-      <inertia ixx="0.0001" ixy="0.0" ixz="0.0"
-        iyy="0.0001" iyz="0.0"
-        izz="0.0001" />
-    </inertial>
-  </link>
-  <joint name="kinect_depth_optical_joint" type="fixed">
-    <origin xyz="0 0 0" rpy="${-M_PI/2} 0 ${-M_PI/2}" />
-    <parent link="kinect_depth_origin" />
-    <child link="kinect_depth" />
-  </joint>
-  <link name="kinect_depth">
-    <inertial>
-      <mass value="0.000001" />
-      <origin xyz="0 0 0" />
-      <inertia ixx="0.0001" ixy="0.0" ixz="0.0"
-        iyy="0.0001" iyz="0.0" izz="0.0001" />
-    </inertial>
-  </link>
-  <joint name="kinect_rgb_joint" type="fixed">
-    <origin xyz="0 -0.005 0" rpy="0 0 0" />
-    <parent link="kinect_link" />
-    <child link="kinect_rgb" />
-  </joint>
-  <link name="kinect_rgb">
-    <inertial>
-      <mass value="0.000001" />
-      <origin xyz="0 0 0" />
-      <inertia ixx="0.0001" ixy="0.0" ixz="0.0"
-        iyy="0.0001" iyz="0.0"
-        izz="0.0001" />
-    </inertial>
-  </link>
-  <!-- ========== synonyms for openni driver ========== -->
-  <joint name="camera_link_joint" type="fixed">
-    <origin xyz="0 0 0" />
-    <parent link="kinect_link" />
-    <child link="camera_link" />
-  </joint>
-  <link name="camera_link">
-    <inertial>
-      <mass value="0.00001" />
-      <origin xyz="0 0 0" />
-      <inertia ixx="1.0" ixy="0.0" ixz="0.0"
-        iyy="1.0" iyz="0.0"
-        izz="1.0" />
-    </inertial>
-  </link>
-  <joint name="camera_depth_joint" type="fixed">
-    <origin xyz="0 0.018 0" rpy="0 0 0" />
-    <parent link="camera_link" />
-    <child link="camera_depth_origin" />
-  </joint>
-  <link name="camera_depth_origin">
-    <inertial>
-      <mass value="0.000001" />
-      <origin xyz="0 0 0" />
-      <inertia ixx="0.0001" ixy="0.0" ixz="0.0"
-        iyy="0.0001" iyz="0.0"
-        izz="0.0001" />
-    </inertial>
-  </link>
-  <joint name="camera_depth_optical_joint" type="fixed">
-    <origin xyz="0 0 0" rpy="${-M_PI/2} 0 ${-M_PI/2}" />
-    <parent link="camera_depth_origin" />
-    <child link="camera_depth" />
-  </joint>
-  <link name="camera_depth">
-    <inertial>
-      <mass value="0.000001" />
-      <origin xyz="0 0 0" />
-      <inertia ixx="0.0001" ixy="0.0" ixz="0.0"
-        iyy="0.0001" iyz="0.0" izz="0.0001" />
-    </inertial>
-  </link>
-  <joint name="camera_rgb_joint" type="fixed">
-    <origin xyz="0 -0.005 0" rpy="0 0 0" />
-    <parent link="camera_link" />
-    <child link="camera_rgb" />
-  </joint>
-  <link name="camera_rgb">
-    <inertial>
-      <mass value="0.000001" />
-      <origin xyz="0 0 0" />
-      <inertia ixx="0.0001" ixy="0.0" ixz="0.0"
-        iyy="0.0001" iyz="0.0"
-        izz="0.0001" />
-    </inertial>
-  </link>
+  <xacro:macro name="kinect" params="camera">
+    <link name="${camera}_link">
+      <inertial>
+        <mass value="0.00001" />
+        <origin xyz="0 0 0" />
+        <inertia ixx="1.0" ixy="0.0" ixz="0.0"
+          iyy="1.0" iyz="0.0"
+          izz="1.0" />
+      </inertial>
+      <visual>
+        <origin xyz="0 0 0" rpy="0 0 0" />
+        <geometry>
+          <mesh filename="package://kurt_description/meshes/kinect/kinect.dae"/>
+        </geometry>
+      </visual>
+      <collision>
+        <origin xyz="-0.0315 0 -0.017" rpy="0 0 0" />
+        <geometry>
+          <box size="0.0730 .2760 0.0720"/>
+        </geometry>
+      </collision>
+    </link>
+    <joint name="${camera}_depth_joint" type="fixed">
+      <origin xyz="0 0.018 0" rpy="0 0 0" />
+      <parent link="kinect_link" />
+      <child link="kinect_depth_origin" />
+    </joint>
+    <link name="${camera}_depth_origin">
+      <inertial>
+        <mass value="0.000001" />
+        <origin xyz="0 0 0" />
+        <inertia ixx="0.0001" ixy="0.0" ixz="0.0"
+          iyy="0.0001" iyz="0.0"
+          izz="0.0001" />
+      </inertial>
+    </link>
+    <joint name="${camera}_depth_optical_joint" type="fixed">
+      <origin xyz="0 0 0" rpy="${-M_PI/2} 0 ${-M_PI/2}" />
+      <parent link="kinect_depth_origin" />
+      <child link="kinect_depth" />
+    </joint>
+    <link name="${camera}_depth">
+      <inertial>
+        <mass value="0.000001" />
+        <origin xyz="0 0 0" />
+        <inertia ixx="0.0001" ixy="0.0" ixz="0.0"
+          iyy="0.0001" iyz="0.0" izz="0.0001" />
+      </inertial>
+    </link>
+    <joint name="${camera}_rgb_joint" type="fixed">
+      <origin xyz="0 -0.005 0" rpy="0 0 0" />
+      <parent link="kinect_link" />
+      <child link="kinect_rgb" />
+    </joint>
+    <link name="${camera}_rgb">
+      <inertial>
+        <mass value="0.000001" />
+        <origin xyz="0 0 0" />
+        <inertia ixx="0.0001" ixy="0.0" ixz="0.0"
+          iyy="0.0001" iyz="0.0"
+          izz="0.0001" />
+      </inertial>
+    </link>
+  </xacro:macro>
 </robot>

File: kurt_description/tops/kurtana_top.urdf.xacro (robot description, xacro)
@@ -14,4 +14,5 @@
   <!-- ************************ -->
   <include filename="$(find kurt_description)/parts/kinect.urdf.xacro" />
+  <xacro:kinect camera="kinect" />
   <joint name="kurtana_kinect_joint" type="fixed">
     <parent link="kurtana_pitchpole_link" />

Commit message: fixed missing occurences of kinect in URDF

File: kurt_description/parts/kinect.urdf.xacro (robot description, xacro)
@@ -30,6 +30,6 @@
     <joint name="${camera}_depth_joint" type="fixed">
       <origin xyz="0 0.018 0" rpy="0 0 0" />
-      <parent link="kinect_link" />
-      <child link="kinect_depth_origin" />
+      <parent link="${camera}_link" />
+      <child link="${camera}_depth_origin" />
     </joint>
     <link name="${camera}_depth_origin">
@@ -44,6 +44,6 @@
     <joint name="${camera}_depth_optical_joint" type="fixed">
       <origin xyz="0 0 0" rpy="${-M_PI/2} 0 ${-M_PI/2}" />
-      <parent link="kinect_depth_origin" />
-      <child link="kinect_depth" />
+      <parent link="${camera}_depth_origin" />
+      <child link="${camera}_depth" />
     </joint>
     <link name="${camera}_depth">
@@ -57,6 +57,6 @@
     <joint name="${camera}_rgb_joint" type="fixed">
       <origin xyz="0 -0.005 0" rpy="0 0 0" />
-      <parent link="kinect_link" />
-      <child link="kinect_rgb" />
+      <parent link="${camera}_link" />
+      <child link="${camera}_rgb" />
     </joint>
     <link name="${camera}_rgb">

Commit message: kinect URDF: changed frame names to match OpenNI driver
this might mean that it doesn't work with old kinect driver any more

File: kurt_description/parts/kinect.urdf.xacro (robot description, xacro)
@@ -31,7 +31,7 @@
       <origin xyz="0 0.018 0" rpy="0 0 0" />
       <parent link="${camera}_link" />
-      <child link="${camera}_depth_origin" />
+      <child link="${camera}_depth_frame" />
     </joint>
-    <link name="${camera}_depth_origin">
+    <link name="${camera}_depth_frame">
       <inertial>
         <mass value="0.000001" />
@@ -44,8 +44,8 @@
     <joint name="${camera}_depth_optical_joint" type="fixed">
       <origin xyz="0 0 0" rpy="${-M_PI/2} 0 ${-M_PI/2}" />
-      <parent link="${camera}_depth_origin" />
-      <child link="${camera}_depth" />
+      <parent link="${camera}_depth_frame" />
+      <child link="${camera}_depth_optical_frame" />
     </joint>
-    <link name="${camera}_depth">
+    <link name="${camera}_depth_optical_frame">
       <inertial>
         <mass value="0.000001" />
@@ -58,7 +58,7 @@
       <origin xyz="0 -0.005 0" rpy="0 0 0" />
       <parent link="${camera}_link" />
-      <child link="${camera}_rgb" />
+      <child link="${camera}_rgb_frame" />
     </joint>
-    <link name="${camera}_rgb">
+    <link name="${camera}_rgb_frame">
       <inertial>
         <mass value="0.000001" />
@@ -69,4 +69,17 @@
       </inertial>
     </link>
+    <joint name="${camera}_rgb_optical_joint" type="fixed">
+      <origin xyz="0 0 0" rpy="${-M_PI/2} 0 ${-M_PI/2}" />
+      <parent link="${camera}_rgb_frame" />
+      <child link="${camera}_rgb_optical_frame" />
+    </joint>
+    <link name="${camera}_rgb_optical_frame">
+      <inertial>
+        <mass value="0.000001" />
+        <origin xyz="0 0 0" />
+        <inertia ixx="0.0001" ixy="0.0" ixz="0.0"
+          iyy="0.0001" iyz="0.0" izz="0.0001" />
+      </inertial>
+    </link>
   </xacro:macro>
 </robot>

Commit message: fix Kinect URDF inertia

File: kurt_description/parts/kinect.urdf.xacro (robot description, xacro)
@@ -5,14 +5,7 @@
   xmlns:xacro="http://ros.org/wiki/xacro"
   name="${camera}">
-  <property name="M_PI" value="3.1415926535897931" />
+  <include filename="$(find kurt_description)/common.xacro" />
   <xacro:macro name="kinect" params="camera">
     <link name="${camera}_link">
-      <inertial>
-        <mass value="0.00001" />
-        <origin xyz="0 0 0" />
-        <inertia ixx="1.0" ixy="0.0" ixz="0.0"
-          iyy="1.0" iyz="0.0"
-          izz="1.0" />
-      </inertial>
       <visual>
         <origin xyz="0 0 0" rpy="0 0 0" />
@@ -24,7 +17,8 @@
         <origin xyz="-0.0315 0 -0.017" rpy="0 0 0" />
         <geometry>
-          <box size="0.0730 .2760 0.0720"/>
+          <box size="0.0730 0.2760 0.0720"/>
         </geometry>
       </collision>
+      <xacro:box_inertial x="0.0730" y="0.2760" z="0.0720" mass="0.430" />
     </link>
     <joint name="${camera}_depth_joint" type="fixed">

Commit message: kinect.urdf.xacro: use mesh from pr2_description
old mesh (from kurt_description) is not shown in either Gazebo or RViz for whatever reason

File: kurt_description/parts/kinect.urdf.xacro (robot description, xacro)
@@ -12,5 +12,5 @@
         <origin xyz="0 0 0" rpy="0 0 0" />
         <geometry>
-          <mesh filename="package://kurt_description/meshes/kinect/kinect.dae"/>
+          <mesh filename="package://pr2_description/meshes/sensors/kinect_v0/kinect.dae" scale="0.001 0.001 0.001" />
         </geometry>
       </visual>
