Commit message: fix indentation

File: kurt_description/parts/kurtana_rack.urdf.xacro (robot description, xacro)
@@ -1,8 +1,8 @@
 <?xml version="1.0"?>
- <robot xmlns:sensor="http://playerstage.sourceforge.net/gazebo/xmlschema/#sensor"
-       xmlns:controller="http://playerstage.sourceforge.net/gazebo/xmlschema/#controller"
-       xmlns:interface="http://playerstage.sourceforge.net/gazebo/xmlschema/#interface"
-       xmlns:xacro="http://ros.org/wiki/xacro"
-       name="kurtana_rack">
+<robot xmlns:sensor="http://playerstage.sourceforge.net/gazebo/xmlschema/#sensor"
+  xmlns:controller="http://playerstage.sourceforge.net/gazebo/xmlschema/#controller"
+  xmlns:interface="http://playerstage.sourceforge.net/gazebo/xmlschema/#interface"
+  xmlns:xacro="http://ros.org/wiki/xacro"
+  name="kurtana_rack">
   <property name="M_PI" value="3.1415926535897931" />
   <!-- all values measured by hand - maybe they need to be optimized later -->
@@ -28,26 +28,26 @@
 <!-- ******************** -->
   <link name="kurtana_rackplate_link">
-      <visual>
-        <origin xyz="0 0 0" rpy="0 0 0" />
-        <geometry>
-          <box size="${rackplate_length} ${rackplate_width} ${rackplate_height}" />
-        </geometry>
-        <material name="grey">
-          <color rgba="0.8 0.8 0.8 1"/>
-        </material>
-      </visual>
-      <collision>
-        <origin xyz="0 0 0" rpy="0 0 0" />
-        <geometry>
-            <box size="${rackplate_length} ${rackplate_width} ${rackplate_height}" />
-        </geometry>
-      </collision>
-      <inertial>
-        <mass value="0.05" />
-        <origin xyz="0.0 0.0 10.0" />
-        <inertia ixx="1.0" ixy="0.0" ixz="0.0"
-                 iyy="1.0" iyz="0.0"
-                 izz="1.0" />
-      </inertial>
+    <visual>
+      <origin xyz="0 0 0" rpy="0 0 0" />
+      <geometry>
+        <box size="${rackplate_length} ${rackplate_width} ${rackplate_height}" />
+      </geometry>
+      <material name="grey">
+        <color rgba="0.8 0.8 0.8 1"/>
+      </material>
+    </visual>
+    <collision>
+      <origin xyz="0 0 0" rpy="0 0 0" />
+      <geometry>
+        <box size="${rackplate_length} ${rackplate_width} ${rackplate_height}" />
+      </geometry>
+    </collision>
+    <inertial>
+      <mass value="0.05" />
+      <origin xyz="0.0 0.0 10.0" />
+      <inertia ixx="1.0" ixy="0.0" ixz="0.0"
+        iyy="1.0" iyz="0.0"
+        izz="1.0" />
+    </inertial>
   </link>
   <joint name="kurtana_baseplate_joint" type="fixed">
@@ -57,37 +57,37 @@
   </joint>
   <link name="kurtana_baseplate_link">
-      <visual>
-        <origin xyz="0 0 0" rpy="0 0 0" />
-        <geometry>
-          <box size="${baseplate_length} ${baseplate_width} ${baseplate_height}" />
-        </geometry>
-        <material name="grey" />
-      </visual>
-      <collision>
-        <origin xyz="0 0 0" rpy="0 0 0" />
-        <geometry>
-          <box size="${baseplate_length} ${baseplate_width} ${baseplate_height}" />
-        </geometry>
-      </collision>
+    <visual>
+      <origin xyz="0 0 0" rpy="0 0 0" />
+      <geometry>
+        <box size="${baseplate_length} ${baseplate_width} ${baseplate_height}" />
+      </geometry>
+      <material name="grey" />
+    </visual>
+    <collision>
+      <origin xyz="0 0 0" rpy="0 0 0" />
+      <geometry>
+        <box size="${baseplate_length} ${baseplate_width} ${baseplate_height}" />
+      </geometry>
+    </collision>
   </link>
-   <joint name="kurtana_pole_joint" type="fixed">
+  <joint name="kurtana_pole_joint" type="fixed">
     <parent link="kurtana_baseplate_link"/>
     <child link="kurtana_pole_link"/>
     <origin xyz="-0.19 0 0"/>
-   </joint>
+  </joint>
   <link name="kurtana_pole_link">
-      <visual>
-        <origin xyz="0 0 ${pole_length/2}" rpy="0 0 0" />
-        <geometry>
-         <cylinder radius="${pole_radius}" length="${pole_length}"/>
-        </geometry>
-        <material name="grey" />
-      </visual>
-      <collision>
-        <origin xyz="0 0 ${pole_length/2}" rpy="0 0 0" />
-        <geometry>
-          <cylinder radius="${pole_radius}" length="${pole_length}"/>
-        </geometry>
-      </collision>
+    <visual>
+      <origin xyz="0 0 ${pole_length/2}" rpy="0 0 0" />
+      <geometry>
+        <cylinder radius="${pole_radius}" length="${pole_length}"/>
+      </geometry>
+      <material name="grey" />
+    </visual>
+    <collision>
+      <origin xyz="0 0 ${pole_length/2}" rpy="0 0 0" />
+      <geometry>
+        <cylinder radius="${pole_radius}" length="${pole_length}"/>
+      </geometry>
+    </collision>
   </link>
   <joint name="kurtana_stretch_joint" type="prismatic">
@@ -99,13 +99,13 @@
     <axis xyz="0 0 1"/>
   </joint>
- <link name="kurtana_poletop_stretch_link">
-        <collision>
-        <origin xyz="0 0 ${poletop_length/2}" rpy="0 0 0" />
-        <geometry>
-         <cylinder radius="${poletop_radius}" length="${poletop_length}"/>
-        </geometry>
-      </collision>
+  <link name="kurtana_poletop_stretch_link">
+    <collision>
+      <origin xyz="0 0 ${poletop_length/2}" rpy="0 0 0" />
+      <geometry>
+        <cylinder radius="${poletop_radius}" length="${poletop_length}"/>
+      </geometry>
+    </collision>
   </link>
-   <joint name="kurtana_roll_joint" type="revolute">
+  <joint name="kurtana_roll_joint" type="revolute">
     <parent link="kurtana_poletop_stretch_link"/>
     <child link="kurtana_poletop_roll_link"/>
@@ -115,19 +115,19 @@
   </joint>
   <link name="kurtana_poletop_roll_link">
-      <visual>
-        <origin xyz="0 0 ${poletop_length/2}" rpy="0 0 0" />
-        <geometry>
-          <cylinder radius="${poletop_radius}" length="${poletop_length}"/>
-        </geometry>
-        <material name="red">
-          <color rgba="0.8 0.5 0.8 1"/>
-        </material>
-      </visual>
-      <collision>
-        <origin xyz="0 0 ${poletop_length/2}" rpy="0 0 0" />
-        <geometry>
-         <cylinder radius="${poletop_radius}" length="${poletop_length}"/>
-        </geometry>
-      </collision>
+    <visual>
+      <origin xyz="0 0 ${poletop_length/2}" rpy="0 0 0" />
+      <geometry>
+        <cylinder radius="${poletop_radius}" length="${poletop_length}"/>
+      </geometry>
+      <material name="red">
+        <color rgba="0.8 0.5 0.8 1"/>
+      </material>
+    </visual>
+    <collision>
+      <origin xyz="0 0 ${poletop_length/2}" rpy="0 0 0" />
+      <geometry>
+        <cylinder radius="${poletop_radius}" length="${poletop_length}"/>
+      </geometry>
+    </collision>
   </link>
   <joint name="kurtana_pitch_joint" type="revolute">
@@ -139,17 +139,17 @@
   </joint>
   <link name="kurtana_pitchpole_link">
-      <visual>
-        <origin rpy="${-M_PI/2} 0 0" xyz="0 0 0"/>
-        <geometry>
-          <cylinder radius="${pitchpole_radius}" length="${pitchpole_length}"/>
-        </geometry>
-        <material name="grey" />
-      </visual>
-      <collision>
-        <origin rpy="${-M_PI/2} 0 0" xyz="0 0 0"/>
-        <geometry>
-         <cylinder radius="${pitchpole_radius}" length="${pitchpole_length}"/>
-        </geometry>
-      </collision>
+    <visual>
+      <origin rpy="${-M_PI/2} 0 0" xyz="0 0 0"/>
+      <geometry>
+        <cylinder radius="${pitchpole_radius}" length="${pitchpole_length}"/>
+      </geometry>
+      <material name="grey" />
+    </visual>
+    <collision>
+      <origin rpy="${-M_PI/2} 0 0" xyz="0 0 0"/>
+      <geometry>
+        <cylinder radius="${pitchpole_radius}" length="${pitchpole_length}"/>
+      </geometry>
+    </collision>
   </link>
 </robot>

Commit message: make kurtana poletop longer

File: kurt_description/parts/kurtana_rack.urdf.xacro (robot description, xacro)
@@ -16,15 +16,13 @@
   <property name="pole_radius" value="0.025"/>
   <property name="pole_length" value="0.70"/>
-  <property name="poletop_radius" value="0.025"/>
-  <property name="poletop_length" value="0.04"/>
+  <property name="poletop_radius" value="0.02"/>
+  <property name="poletop_length" value="0.555"/>
+  <property name="poletop_z_offset" value="0.04"/>
   <property name="pitchpole_radius" value="0.012"/>
   <property name="pitchpole_length" value="0.23"/>
-  <property name="kinect_length" value="0.30" />
-  <property name="kinect_width" value="0.08" />
-  <property name="kinect_height" value="0.08" />
   <property name="kinect_gap" value="0.015" />
-<!-- ******************** -->
-<!-- *** KURTana Rack *** -->
-<!-- ******************** -->
+  <!-- ******************** -->
+  <!-- *** KURTana Rack *** -->
+  <!-- ******************** -->
   <link name="kurtana_rackplate_link">
     <visual>
@@ -95,15 +93,8 @@
     <child link="kurtana_poletop_stretch_link"/>
     <origin xyz="0 0 ${pole_length}" rpy="0 0 0"/>
-    <limit effort="1000.0" lower="0" upper="0.515" velocity="0.5"/>
-    <origin rpy="0 0 0" xyz="0 0 0"/>
+    <limit effort="1000.0" lower="0" upper="${poletop_length - poletop_z_offset}" velocity="0.5"/>
     <axis xyz="0 0 1"/>
   </joint>
   <link name="kurtana_poletop_stretch_link">
-    <collision>
-      <origin xyz="0 0 ${poletop_length/2}" rpy="0 0 0" />
-      <geometry>
-        <cylinder radius="${poletop_radius}" length="${poletop_length}"/>
-      </geometry>
-    </collision>
   </link>
   <joint name="kurtana_roll_joint" type="revolute">
@@ -116,14 +107,12 @@
   <link name="kurtana_poletop_roll_link">
     <visual>
-      <origin xyz="0 0 ${poletop_length/2}" rpy="0 0 0" />
+      <origin xyz="0 0 ${poletop_z_offset - poletop_length/2}" rpy="0 0 0" />
       <geometry>
         <cylinder radius="${poletop_radius}" length="${poletop_length}"/>
       </geometry>
-      <material name="red">
-        <color rgba="0.8 0.5 0.8 1"/>
-      </material>
+      <material name="grey" />
     </visual>
     <collision>
-      <origin xyz="0 0 ${poletop_length/2}" rpy="0 0 0" />
+      <origin xyz="0 0 ${poletop_z_offset - poletop_length/2}" rpy="0 0 0" />
       <geometry>
         <cylinder radius="${poletop_radius}" length="${poletop_length}"/>
@@ -134,5 +123,5 @@
     <parent link="kurtana_poletop_roll_link" />
     <child link="kurtana_pitchpole_link" />
-    <origin xyz="0 0 ${poletop_length/2}" rpy="0 0 0"/>
+    <origin xyz="0 0 ${poletop_z_offset/2}" rpy="0 0 0"/>
     <axis xyz="0 1 0"/>
     <limit effort="1000.0" lower="${-M_PI/2}" upper="${M_PI/2}" velocity="2.0"/>

Commit message: shift URDF origins to make link + visual match
makes including proper inertials later much easier

File: kurt_description/parts/kurtana_rack.urdf.xacro (robot description, xacro)
@@ -72,9 +72,9 @@
     <parent link="kurtana_baseplate_link"/>
     <child link="kurtana_pole_link"/>
-    <origin xyz="-0.19 0 0"/>
+    <origin xyz="-0.19 0 ${pole_length/2}"/>
   </joint>
   <link name="kurtana_pole_link">
     <visual>
-      <origin xyz="0 0 ${pole_length/2}" rpy="0 0 0" />
+      <origin xyz="0 0 0" rpy="0 0 0" />
       <geometry>
         <cylinder radius="${pole_radius}" length="${pole_length}"/>
@@ -83,5 +83,5 @@
     </visual>
     <collision>
-      <origin xyz="0 0 ${pole_length/2}" rpy="0 0 0" />
+      <origin xyz="0 0 0" rpy="0 0 0" />
       <geometry>
         <cylinder radius="${pole_radius}" length="${pole_length}"/>
@@ -92,5 +92,5 @@
     <parent link="kurtana_pole_link"/>
     <child link="kurtana_poletop_stretch_link"/>
-    <origin xyz="0 0 ${pole_length}" rpy="0 0 0"/>
+    <origin xyz="0 0 ${poletop_z_offset + pole_length/2 - poletop_length/2}" rpy="0 0 0"/>
     <limit effort="1000.0" lower="0" upper="${poletop_length - poletop_z_offset}" velocity="0.5"/>
     <axis xyz="0 0 1"/>
@@ -107,5 +107,5 @@
   <link name="kurtana_poletop_roll_link">
     <visual>
-      <origin xyz="0 0 ${poletop_z_offset - poletop_length/2}" rpy="0 0 0" />
+      <origin xyz="0 0 0" rpy="0 0 0" />
       <geometry>
         <cylinder radius="${poletop_radius}" length="${poletop_length}"/>
@@ -114,5 +114,5 @@
     </visual>
     <collision>
-      <origin xyz="0 0 ${poletop_z_offset - poletop_length/2}" rpy="0 0 0" />
+      <origin xyz="0 0 0" rpy="0 0 0" />
       <geometry>
         <cylinder radius="${poletop_radius}" length="${poletop_length}"/>
@@ -123,5 +123,5 @@
     <parent link="kurtana_poletop_roll_link" />
     <child link="kurtana_pitchpole_link" />
-    <origin xyz="0 0 ${poletop_z_offset/2}" rpy="0 0 0"/>
+    <origin xyz="0 0 ${poletop_length/2 - poletop_z_offset/2}" rpy="0 0 0"/>
     <axis xyz="0 1 0"/>
     <limit effort="1000.0" lower="${-M_PI/2}" upper="${M_PI/2}" velocity="2.0"/>

Commit message: remeasured kurtana rack URDFs, now fit perfectly

File: kurt_description/parts/kurtana_rack.urdf.xacro (robot description, xacro)
@@ -7,8 +7,8 @@
   <property name="M_PI" value="3.1415926535897931" />
   <!-- all values measured by hand - maybe they need to be optimized later -->
-  <property name="rackplate_length" value="0.51" />
+  <property name="rackplate_length" value="0.47" />
   <property name="rackplate_width" value="0.368" />
   <property name="rackplate_height" value="0.023" />
-  <property name="baseplate_length" value="0.51" />
+  <property name="baseplate_length" value="0.47" />
   <property name="baseplate_width" value="0.368" />
   <property name="baseplate_height" value="0.005" />
@@ -16,4 +16,5 @@
   <property name="pole_radius" value="0.025"/>
   <property name="pole_length" value="0.70"/>
+  <property name="pole_x_offset" value="-0.165"/>
   <property name="poletop_radius" value="0.02"/>
   <property name="poletop_length" value="0.555"/>
@@ -21,8 +22,8 @@
   <property name="pitchpole_radius" value="0.012"/>
   <property name="pitchpole_length" value="0.23"/>
-  <property name="kinect_gap" value="0.015" />
   <!-- ******************** -->
   <!-- *** KURTana Rack *** -->
   <!-- ******************** -->
+  <!-- rackplate = lower plate-->
   <link name="kurtana_rackplate_link">
     <visual>
@@ -49,8 +50,9 @@
     </inertial>
   </link>
+  <!-- baseplate = upper plate -->
   <joint name="kurtana_baseplate_joint" type="fixed">
     <parent link="kurtana_rackplate_link"/>
     <child link="kurtana_baseplate_link"/>
-    <origin xyz="0 0 0.055"/>
+    <origin xyz="0 0 ${rackplate_height/2 + rackgap + baseplate_height/2}"/>
   </joint>
   <link name="kurtana_baseplate_link">
@@ -69,8 +71,9 @@
     </collision>
   </link>
+  <!-- pole = lower, fixed, hollow pole -->
   <joint name="kurtana_pole_joint" type="fixed">
     <parent link="kurtana_baseplate_link"/>
     <child link="kurtana_pole_link"/>
-    <origin xyz="-0.19 0 ${pole_length/2}"/>
+    <origin xyz="${pole_x_offset} 0 ${pole_length/2}"/>
   </joint>
   <link name="kurtana_pole_link">
@@ -89,4 +92,5 @@
     </collision>
   </link>
+  <!-- poletop = upper, inner, moving pole -->
   <joint name="kurtana_stretch_joint" type="prismatic">
     <parent link="kurtana_pole_link"/>
@@ -120,4 +124,5 @@
     </collision>
   </link>
+  <!-- pitchpole = horizontal pole on top where kinect is mounted -->
   <joint name="kurtana_pitch_joint" type="revolute">
     <parent link="kurtana_poletop_roll_link" />

File: kurt_description/tops/kurtana_top.urdf.xacro (robot description, xacro)
@@ -10,4 +10,6 @@
   <!-- ******************** -->
   <include filename="$(find kurt_description)/parts/kurtana_rack.urdf.xacro" />
+  <property name="kinect_x_offset" value="0.025" />
+  <property name="kinect_z_offset" value="0.087" />
   <!-- ************************ -->
   <!-- *** Microsoft Kinect *** -->
@@ -18,5 +20,5 @@
     <parent link="kurtana_pitchpole_link" />
     <child  link="kinect_link" />
-    <origin xyz="${0.0730/2} 0 ${0.0720+kinect_gap}" rpy="0 0 0"/>
+    <origin xyz="${kinect_x_offset} 0 ${kinect_z_offset}" rpy="0 0 0"/>
   </joint>
   <!-- **************************** -->

Commit message: fixed kurtana description

File: kurt_description/parts/kurtana_rack.urdf.xacro (robot description, xacro)
@@ -12,9 +12,9 @@
   <property name="baseplate_length" value="0.47" />
   <property name="baseplate_width" value="0.368" />
-  <property name="baseplate_height" value="0.005" />
+  <property name="baseplate_height" value="0.006" />
   <property name="rackgap" value="0.055" />
   <property name="pole_radius" value="0.025"/>
   <property name="pole_length" value="0.70"/>
-  <property name="pole_x_offset" value="-0.165"/>
+  <property name="pole_x_offset" value="-0.15"/>
   <property name="poletop_radius" value="0.02"/>
   <property name="poletop_length" value="0.555"/>

File: kurt_description/robots/kurtana.urdf.xacro (robot description, xacro)
@@ -3,6 +3,6 @@
   xmlns:xacro="http://ros.org/wiki/xacro"
   name="kurt360">
-  <xacro:property name="top_y_offset" value="0.009" />
-  <xacro:property name="base_z_offset" value="0.03" /> <!-- distance from base_link to top of cover surface -->
+  <xacro:property name="top_y_offset" value="0.00" />
+  <xacro:property name="base_z_offset" value="0.012" /> <!-- distance from base_link to top of cover surface -->
   <include filename="$(find kurt_description)/bases/kurt_outdoor.urdf.xacro" />
   <include filename="$(find kurt_description)/tops/kurtana_top.urdf.xacro" />

File: kurt_description/tops/kurtana_top.urdf.xacro (robot description, xacro)
@@ -10,5 +10,5 @@
   <!-- ******************** -->
   <include filename="$(find kurt_description)/parts/kurtana_rack.urdf.xacro" />
-  <property name="kinect_x_offset" value="0.025" />
+  <property name="kinect_x_offset" value="0.018" />
   <property name="kinect_z_offset" value="0.087" />
   <!-- ************************ -->
