Commit message: made kurtana URDF gazebo-ready
- added inertials to kurtana URDF (necessary for gazebo)
- switched stretch and roll link (it's much better in gazebo when the long sliding shaft is the prismatic
link)
- renamed poletop to innerpole, made proper poletop
- added transmissions

File: kurt_description/parts/kurtana_rack.urdf.xacro (robot description, xacro)
@@ -5,21 +5,28 @@
   xmlns:xacro="http://ros.org/wiki/xacro"
   name="kurtana_rack">
-  <property name="M_PI" value="3.1415926535897931" />
-  <!-- all values measured by hand - maybe they need to be optimized later -->
+  <include filename="$(find kurt_description)/common.xacro" />
   <property name="rackplate_length" value="0.47" />
   <property name="rackplate_width" value="0.368" />
   <property name="rackplate_height" value="0.023" />
+  <property name="rackplate_mass" value="0.500" />
   <property name="baseplate_length" value="0.47" />
   <property name="baseplate_width" value="0.368" />
   <property name="baseplate_height" value="0.006" />
+  <property name="baseplate_mass" value="0.500" />
   <property name="rackgap" value="0.055" />
   <property name="pole_radius" value="0.025"/>
   <property name="pole_length" value="0.70"/>
   <property name="pole_x_offset" value="-0.15"/>
-  <property name="poletop_radius" value="0.02"/>
-  <property name="poletop_length" value="0.555"/>
-  <property name="poletop_z_offset" value="0.04"/>
+  <property name="pole_mass" value="3.0"/>
+  <property name="innerpole_radius" value="0.02"/>
+  <property name="innerpole_length" value="0.555"/>
+  <property name="innerpole_z_offset" value="0.04"/>
+  <property name="innerpole_mass" value="2.0"/>
+  <property name="poletop_radius" value="0.025"/>
+  <property name="poletop_length" value="0.04"/>
+  <property name="poletop_mass" value="0.1"/>
   <property name="pitchpole_radius" value="0.012"/>
   <property name="pitchpole_length" value="0.23"/>
+  <property name="pitchpole_mass" value="0.050"/>
   <!-- ******************** -->
   <!-- *** KURTana Rack *** -->
@@ -42,11 +49,5 @@
       </geometry>
     </collision>
-    <inertial>
-      <mass value="0.05" />
-      <origin xyz="0.0 0.0 10.0" />
-      <inertia ixx="1.0" ixy="0.0" ixz="0.0"
-        iyy="1.0" iyz="0.0"
-        izz="1.0" />
-    </inertial>
+    <xacro:box_inertial x="${rackplate_length}" y="${rackplate_width}" z="${rackplate_height}" mass="${rackplate_mass}" />
   </link>
   <!-- baseplate = upper plate -->
@@ -70,4 +71,5 @@
       </geometry>
     </collision>
+    <xacro:box_inertial x="${baseplate_length}" y="${baseplate_width}" z="${baseplate_height}" mass="${baseplate_mass}" />
   </link>
   <!-- pole = lower, fixed, hollow pole -->
@@ -91,19 +93,34 @@
       </geometry>
     </collision>
-  </link>
-  <!-- poletop = upper, inner, moving pole -->
+    <xacro:cylinder_inertial radius="${pole_radius}" length="${pole_length}" mass="${pole_mass}" />
+  </link>
+  <!-- innerpole = upper, inner, moving pole -->
   <joint name="kurtana_stretch_joint" type="prismatic">
     <parent link="kurtana_pole_link"/>
-    <child link="kurtana_poletop_stretch_link"/>
-    <origin xyz="0 0 ${poletop_z_offset + pole_length/2 - poletop_length/2}" rpy="0 0 0"/>
-    <limit effort="1000.0" lower="0" upper="${poletop_length - poletop_z_offset}" velocity="0.5"/>
+    <child link="kurtana_innerpole_stretch_link"/>
+    <origin xyz="0 0 ${innerpole_z_offset + pole_length/2 - innerpole_length/2}" rpy="0 0 0"/>
+    <limit effort="1000.0" lower="0" upper="${innerpole_length - innerpole_z_offset}" velocity="0.5"/>
     <axis xyz="0 0 1"/>
   </joint>
-  <link name="kurtana_poletop_stretch_link">
+  <link name="kurtana_innerpole_stretch_link">
+    <visual>
+      <origin xyz="0 0 0" rpy="0 0 0" />
+      <geometry>
+        <cylinder radius="${innerpole_radius}" length="${innerpole_length}"/>
+      </geometry>
+      <material name="grey" />
+    </visual>
+    <collision>
+      <origin xyz="0 0 0" rpy="0 0 0" />
+      <geometry>
+        <cylinder radius="${innerpole_radius}" length="${innerpole_length}"/>
+      </geometry>
+    </collision>
+    <xacro:cylinder_inertial radius="${innerpole_radius}" length="${innerpole_length}" mass="${innerpole_mass}" />
   </link>
   <joint name="kurtana_roll_joint" type="revolute">
-    <parent link="kurtana_poletop_stretch_link"/>
+    <parent link="kurtana_innerpole_stretch_link"/>
     <child link="kurtana_poletop_roll_link"/>
-    <origin xyz="0 0 0" rpy="0 0 0"/>
+    <origin xyz="0 0 ${innerpole_length/2 - innerpole_z_offset/2}" rpy="0 0 0"/>
     <axis xyz="0 0 1"/>
     <limit effort="1000.0" lower="${-M_PI/2}" upper="${M_PI/2}" velocity="2.0"/>
@@ -123,4 +140,5 @@
       </geometry>
     </collision>
+    <xacro:cylinder_inertial radius="${poletop_radius}" length="${poletop_length}" mass="${poletop_mass}" />
   </link>
   <!-- pitchpole = horizontal pole on top where kinect is mounted -->
@@ -128,5 +146,5 @@
     <parent link="kurtana_poletop_roll_link" />
     <child link="kurtana_pitchpole_link" />
-    <origin xyz="0 0 ${poletop_length/2 - poletop_z_offset/2}" rpy="0 0 0"/>
+    <origin xyz="0 0 0" rpy="0 0 0"/>
     <axis xyz="0 1 0"/>
     <limit effort="1000.0" lower="${-M_PI/2}" upper="${M_PI/2}" velocity="2.0"/>
@@ -146,4 +164,38 @@
       </geometry>
     </collision>
-  </link>
+    <xacro:cylinder_inertial radius="${pitchpole_radius}" length="${pitchpole_length}" mass="${pitchpole_mass}" />
+  </link>
+  <!-- ******************** -->
+  <!-- *** Gazebo stuff *** -->
+  <!-- ******************** -->
+  <!-- transmissions are required by the controller manager (here: for simulation in gazebo) -->
+  <xacro:macro name="kurtana_pole_transmission" params="name">
+    <transmission name="${name}_trans" type="pr2_mechanism_model/SimpleTransmission">
+      <actuator name="${name}_motor" />
+      <joint name="${name}_joint" />
+      <mechanicalReduction>1</mechanicalReduction>
+      <motorTorqueConstant>1</motorTorqueConstant>
+    </transmission>
+  </xacro:macro>
+  <xacro:kurtana_pole_transmission name="kurtana_stretch" />
+  <xacro:kurtana_pole_transmission name="kurtana_roll" />
+  <xacro:kurtana_pole_transmission name="kurtana_pitch" />
+  <gazebo reference="kurtana_rackplate_link">
+    <material value="PR2/Grey1" />
+  </gazebo>
+  <gazebo reference="kurtana_baseplate_link">
+    <material value="PR2/Grey1" />
+  </gazebo>
+  <gazebo reference="kurtana_pole_link">
+    <material value="PR2/Grey1" />
+  </gazebo>
+  <gazebo reference="kurtana_innerpole_stretch_link">
+    <material value="PR2/Grey1" />
+  </gazebo>
+  <gazebo reference="kurtana_poletop_roll_link">
+    <material value="PR2/Grey1" />
+  </gazebo>
+  <gazebo reference="kurtana_pitchpole_link">
+    <material value="PR2/Grey1" />
+  </gazebo>
 </robot>

Commit message: fix kurtana colors in gazebo

File: kurt_description/parts/kurtana_rack.urdf.xacro (robot description, xacro)
@@ -182,20 +182,20 @@
   <xacro:kurtana_pole_transmission name="kurtana_pitch" />
   <gazebo reference="kurtana_rackplate_link">
-    <material value="PR2/Grey1" />
+    <material value="PR2/Grey" />
   </gazebo>
   <gazebo reference="kurtana_baseplate_link">
-    <material value="PR2/Grey1" />
+    <material value="PR2/Grey" />
   </gazebo>
   <gazebo reference="kurtana_pole_link">
-    <material value="PR2/Grey1" />
+    <material value="PR2/Grey" />
   </gazebo>
   <gazebo reference="kurtana_innerpole_stretch_link">
-    <material value="PR2/Grey1" />
+    <material value="PR2/Grey" />
   </gazebo>
   <gazebo reference="kurtana_poletop_roll_link">
-    <material value="PR2/Grey1" />
+    <material value="PR2/Grey" />
   </gazebo>
   <gazebo reference="kurtana_pitchpole_link">
-    <material value="PR2/Grey1" />
+    <material value="PR2/Grey" />
   </gazebo>
 </robot>
