Commit message: Add IR and sonar to URDF.

File: kurt_description/bases/kurt_indoor.urdf.xacro (robot description, xacro)
@@ -5,5 +5,6 @@
   xmlns:xacro="http://ros.org/wiki/xacro"
   name="kurt_outdoor_base">
-  <xacro:property name="PI" value="3.14159" />
+  <include filename="$(find kurt_description)/common.xacro" />
+  <include filename="$(find kurt_description)/parts/infrared_sonar.urdf.xacro" />
   <!-- TODO: measure all these values on a real KURT -->
   <xacro:property name="wheel_width" value="0.02" />
@@ -82,5 +83,5 @@
     <link name="${name}_wheel_link">
       <visual>
-        <origin xyz="0 0 0" rpy="0 0 ${rotate_visual * PI}" />
+        <origin xyz="0 0 0" rpy="0 0 ${rotate_visual * M_PI}" />
         <geometry>
           <mesh filename="package://kurt_description/meshes/kurt_wheel_indoor.dae" />

File: kurt_description/bases/kurt_outdoor.urdf.xacro (robot description, xacro)
@@ -5,5 +5,6 @@
   xmlns:xacro="http://ros.org/wiki/xacro"
   name="kurt_outdoor_base">
-  <xacro:property name="PI" value="3.14159" />
+  <include filename="$(find kurt_description)/common.xacro" />
+  <include filename="$(find kurt_description)/parts/infrared_sonar.urdf.xacro" />
   <!-- TODO: measure all these values on a real KURT -->
   <xacro:property name="wheel_width" value="0.04" />

Commit message: increased weight of kurt base in gazebo to real value

File: kurt_description/bases/kurt_indoor.urdf.xacro (robot description, xacro)
@@ -15,4 +15,5 @@
   <xacro:property name="wheel_z_offset" value="-0.10" />
   <xacro:property name="turning_adaptation" value="0.60" />  <!-- physical kurt indoor: 0.69 -->
+  <xacro:property name="mass" value="15.6" />
   <link name="base_link">
     <visual>
@@ -40,9 +41,9 @@
     </visual> -->
     <inertial>
-      <mass value="7.0" />
+      <mass value="${mass}" />
       <origin xyz="0.0 0.0 -0.040426445" />
-      <inertia ixx="0.053184933" ixy="0.0" ixz="0.0"
-        iyy="0.086499893" iyz="0.0"
-        izz="0.107785706" />
+      <inertia ixx="${mass * 0.007597848}" ixy="0.0" ixz="0.0"
+        iyy="${mass * 0.012357128}" iyz="0.0"
+        izz="${mass * 0.015397958}" />
     </inertial>
   </link>

File: kurt_description/bases/kurt_outdoor.urdf.xacro (robot description, xacro)
@@ -15,4 +15,5 @@
   <xacro:property name="wheel_z_offset" value="-0.10" />
   <xacro:property name="turning_adaptation" value="0.60" />  <!-- physical kurt outdoor: 0.46 -->
+  <xacro:property name="mass" value="15.6" />
   <link name="base_link">
     <visual>
@@ -40,9 +41,9 @@
     </visual> -->
     <inertial>
-      <mass value="7.0" />
+      <mass value="${mass}" />
       <origin xyz="0.0 0.0 -0.040426445" />
-      <inertia ixx="0.053184933" ixy="0.0" ixz="0.0"
-        iyy="0.086499893" iyz="0.0"
-        izz="0.107785706" />
+      <inertia ixx="${mass * 0.007597848}" ixy="0.0" ixz="0.0"
+        iyy="${mass * 0.012357128}" iyz="0.0"
+        izz="${mass * 0.015397958}" />
     </inertial>
   </link>

Commit message: add IMU to Kurt model in Gazebo

File: kurt_description/bases/kurt_indoor.urdf.xacro (robot description, xacro)
@@ -7,4 +7,5 @@
   <include filename="$(find kurt_description)/common.xacro" />
   <include filename="$(find kurt_description)/parts/infrared_sonar.urdf.xacro" />
+  <include filename="$(find kurt_description)/parts/imu.gazebo.urdf.xacro" />
   <!-- TODO: measure all these values on a real KURT -->
   <xacro:property name="wheel_width" value="0.02" />
@@ -16,4 +17,5 @@
   <xacro:property name="turning_adaptation" value="0.60" />  <!-- physical kurt indoor: 0.69 -->
   <xacro:property name="mass" value="15.6" />
+  <xacro:property name="imu_stdev" value="0.00017" />
   <link name="base_link">
     <visual>
@@ -80,4 +82,6 @@
     </controller:gazebo_ros_p3d>
   </gazebo>
+  <!-- inertial measurement unit for gazebo -->
+  <xacro:imu_gazebo link="base_link" imu_topic="imu" update_rate="100.0" stdev="${imu_stdev}" />
   <xacro:macro name="kurt_wheel" params="name xyz rotate_visual">
     <!-- rotate_visual: 0 for right side, 1 for left side -->

File: kurt_description/bases/kurt_outdoor.urdf.xacro (robot description, xacro)
@@ -7,4 +7,5 @@
   <include filename="$(find kurt_description)/common.xacro" />
   <include filename="$(find kurt_description)/parts/infrared_sonar.urdf.xacro" />
+  <include filename="$(find kurt_description)/parts/imu.gazebo.urdf.xacro" />
   <!-- TODO: measure all these values on a real KURT -->
   <xacro:property name="wheel_width" value="0.04" />
@@ -16,4 +17,5 @@
   <xacro:property name="turning_adaptation" value="0.60" />  <!-- physical kurt outdoor: 0.46 -->
   <xacro:property name="mass" value="15.6" />
+  <xacro:property name="imu_stdev" value="0.00017" />
   <link name="base_link">
     <visual>
@@ -80,4 +82,6 @@
     </controller:gazebo_ros_p3d>
   </gazebo>
+  <!-- inertial measurement unit for gazebo -->
+  <xacro:imu_gazebo link="base_link" imu_topic="imu" update_rate="100.0" stdev="${imu_stdev}" />
   <xacro:macro name="kurt_wheel" params="name xyz">
     <link name="${name}_wheel_link">

Commit message: using STL files for collision instead of DAE
fixes http://answers.ros.org/question/2368/gazebo-model-wheels-slip-after-upgrade-to-electric

not strictly necessary for the wheels, but better be safe

File: kurt_description/bases/kurt_indoor.urdf.xacro (robot description, xacro)
@@ -97,5 +97,6 @@
         <origin xyz="0 0 0" rpy="0 0 0" />
         <geometry>
-          <mesh filename="package://kurt_description/meshes/kurt_wheel_indoor.dae" />
+          <!-- using STL for collision to fix http://answers.ros.org/question/2368/gazebo-model-wheels-slip-after-upgrade-to-electric -->
+          <mesh filename="package://kurt_description/meshes/kurt_wheel_indoor.stl" />
           <!-- <cylinder length="${wheel_width}" radius="${wheel_radius}" /> -->
         </geometry>

File: kurt_description/tops/kurt2.urdf.xacro (robot description, xacro)
@@ -11,5 +11,6 @@
     <collision>
       <geometry>
-        <mesh filename="package://kurt_description/meshes/laptop_structure.dae" />
+        <!-- using STL for collision to fix http://answers.ros.org/question/2368/gazebo-model-wheels-slip-after-upgrade-to-electric -->
+        <mesh filename="package://kurt_description/meshes/laptop_structure.stl" />
       </geometry>
     </collision>

Commit message: copy axis_length etc from physical kurt to simulated

File: kurt_description/bases/kurt_indoor.urdf.xacro (robot description, xacro)
@@ -10,10 +10,10 @@
   <!-- TODO: measure all these values on a real KURT -->
   <xacro:property name="wheel_width" value="0.02" />
-  <xacro:property name="wheel_radius" value="0.060319723" />
-  <xacro:property name="axis_length" value="0.26" />
-  <xacro:property name="middle_axis_length" value="0.26" />
+  <xacro:property name="wheel_radius" value="0.060319723" /> <!-- from physical kurt_outdoor (corresponds to wheel_perimeter=0.379) -->
+  <xacro:property name="axis_length" value="0.28" /> <!-- from physical kurt_indoor -->
+  <xacro:property name="middle_axis_length" value="0.28" /> <!-- from physical kurt_indoor -->
   <xacro:property name="wheel_x_offset" value="0.13" />
   <xacro:property name="wheel_z_offset" value="-0.10" />
-  <xacro:property name="turning_adaptation" value="0.60" />  <!-- physical kurt indoor: 0.69 -->
+  <xacro:property name="turning_adaptation" value="0.69" />  <!-- from physical kurt_indoor -->
   <xacro:property name="mass" value="15.6" />
   <xacro:property name="imu_stdev" value="0.00017" />

File: kurt_description/bases/kurt_outdoor.urdf.xacro (robot description, xacro)
@@ -10,10 +10,10 @@
   <!-- TODO: measure all these values on a real KURT -->
   <xacro:property name="wheel_width" value="0.04" />
-  <xacro:property name="wheel_radius" value="0.08244" />
+  <xacro:property name="wheel_radius" value="0.08244" /> <!-- from physical kurt_outdoor (corresponds to wheel_perimeter=0.518) -->
   <xacro:property name="axis_length" value="0.28" />
-  <xacro:property name="middle_axis_length" value="0.37" />
+  <xacro:property name="middle_axis_length" value="0.39" /> <!-- from physical kurt_outdoor -->
   <xacro:property name="wheel_x_offset" value="0.14" />
   <xacro:property name="wheel_z_offset" value="-0.10" />
-  <xacro:property name="turning_adaptation" value="0.60" />  <!-- physical kurt outdoor: 0.46 -->
+  <xacro:property name="turning_adaptation" value="0.64" /> <!-- from physical kurt_outdoor -->
   <xacro:property name="mass" value="15.6" />
   <xacro:property name="imu_stdev" value="0.00017" />

Commit message: measured URDF values on physical Kurt (bases)

File: kurt_description/bases/kurt_indoor.urdf.xacro (robot description, xacro)
@@ -8,12 +8,11 @@
   <include filename="$(find kurt_description)/parts/infrared_sonar.urdf.xacro" />
   <include filename="$(find kurt_description)/parts/imu.gazebo.urdf.xacro" />
-  <!-- TODO: measure all these values on a real KURT -->
-  <xacro:property name="wheel_width" value="0.02" />
-  <xacro:property name="wheel_radius" value="0.060319723" /> <!-- from physical kurt_outdoor (corresponds to wheel_perimeter=0.379) -->
-  <xacro:property name="axis_length" value="0.28" /> <!-- from physical kurt_indoor -->
-  <xacro:property name="middle_axis_length" value="0.28" /> <!-- from physical kurt_indoor -->
-  <xacro:property name="wheel_x_offset" value="0.13" />
-  <xacro:property name="wheel_z_offset" value="-0.10" />
-  <xacro:property name="turning_adaptation" value="0.69" />  <!-- from physical kurt_indoor -->
+  <xacro:property name="wheel_width" value="0.035" />
+  <xacro:property name="wheel_radius" value="0.060319723" /> <!-- corresponds to wheel_perimeter=0.379 -->
+  <xacro:property name="axis_length" value="0.28" />
+  <xacro:property name="middle_axis_length" value="0.28" />
+  <xacro:property name="wheel_x_offset" value="0.14" />
+  <xacro:property name="wheel_z_offset" value="-0.107" />
+  <xacro:property name="turning_adaptation" value="0.69" />
   <xacro:property name="mass" value="15.6" />
   <xacro:property name="imu_stdev" value="0.00017" />

File: kurt_description/bases/kurt_outdoor.urdf.xacro (robot description, xacro)
@@ -8,12 +8,11 @@
   <include filename="$(find kurt_description)/parts/infrared_sonar.urdf.xacro" />
   <include filename="$(find kurt_description)/parts/imu.gazebo.urdf.xacro" />
-  <!-- TODO: measure all these values on a real KURT -->
-  <xacro:property name="wheel_width" value="0.04" />
-  <xacro:property name="wheel_radius" value="0.08244" /> <!-- from physical kurt_outdoor (corresponds to wheel_perimeter=0.518) -->
+  <xacro:property name="wheel_width" value="0.046" />
+  <xacro:property name="wheel_radius" value="0.08244" /> <!-- corresponds to wheel_perimeter=0.518 -->
   <xacro:property name="axis_length" value="0.28" />
-  <xacro:property name="middle_axis_length" value="0.39" /> <!-- from physical kurt_outdoor -->
+  <xacro:property name="middle_axis_length" value="0.39" />
   <xacro:property name="wheel_x_offset" value="0.14" />
-  <xacro:property name="wheel_z_offset" value="-0.10" />
-  <xacro:property name="turning_adaptation" value="0.64" /> <!-- from physical kurt_outdoor -->
+  <xacro:property name="wheel_z_offset" value="-0.107" />
+  <xacro:property name="turning_adaptation" value="0.64" />
   <xacro:property name="mass" value="15.6" />
   <xacro:property name="imu_stdev" value="0.00017" />

Commit message: converted some URDFs to new SDF 1.5 compatible format
thanks to Michael Görner

File: kurt_description/bases/kurt_indoor.urdf.xacro (robot description, xacro)
@@ -53,5 +53,5 @@
   </gazebo>
   <gazebo>
-    <controller:gazebo_ros_kurt name="kurt_controller" plugin="libgazebo_ros_kurt.so">
+    <plugin name="kurt_controller" filename="libgazebo_ros_kurt.so">
       <alwaysOn>true</alwaysOn>
       <cmd_vel_topic_name>cmd_vel</cmd_vel_topic_name>
@@ -70,9 +70,9 @@
       <max_velocity>0.9</max_velocity>
       <updateRate>40.0</updateRate>
-    </controller:gazebo_ros_kurt>
+    </plugin>
   </gazebo>
   <!-- publish ground truth for pose of base_footprint -->
   <gazebo>
-    <controller:gazebo_ros_p3d name="base_footprint_controller" plugin="libgazebo_ros_p3d.so">
+    <plugin name="base_footprint_controller" filename="libgazebo_ros_p3d.so">
       <alwaysOn>true</alwaysOn>
       <updateRate>30.0</updateRate>
@@ -82,5 +82,5 @@
       <frameName>map</frameName>
       <interface:position name="base_footprint_p3d_position_iface" />
-    </controller:gazebo_ros_p3d>
+    </plugin>
   </gazebo>
   <!-- inertial measurement unit for gazebo -->

File: kurt_description/parts/imu.gazebo.urdf.xacro (robot description, xacro)
@@ -5,5 +5,5 @@
   <xacro:macro name="imu_gazebo" params="link imu_topic update_rate stdev">
     <gazebo>
-      <controller:gazebo_ros_imu name="imu_controller" plugin="libgazebo_ros_imu.so">
+      <plugin name="imu_controller" filename="libgazebo_ros_imu.so">
         <alwaysOn>true</alwaysOn>
         <updateRate>${update_rate}</updateRate>
@@ -14,5 +14,5 @@
         <rpyOffsets>0 0 0</rpyOffsets>
         <interface:position name="imu_position"/>
-      </controller:gazebo_ros_imu>
+      </plugin>
     </gazebo>
   </xacro:macro>

File: kurt_description/parts/sick_lms200.urdf.xacro (robot description, xacro)
@@ -29,25 +29,31 @@
   <gazebo reference="laser">
     <material value="Gazebo/Blue" />
-    <sensor:ray name="laser">
-      <rayCount>181</rayCount>
-      <rangeCount>181</rangeCount>
-      <laserCount>1</laserCount>
-      <origin>0.0 0.0 0.0</origin>
-      <displayRays>false</displayRays>
-      <minAngle>-90</minAngle>
-      <maxAngle>90</maxAngle>
-      <minRange>0.08</minRange>
-      <maxRange>10.0</maxRange>
-      <resRange>0.01</resRange>
-      <updateRate>75.0</updateRate>
-      <controller:gazebo_ros_laser name="gazebo_ros_laser_controller" plugin="libgazebo_ros_laser.so">
+    <sensor type="ray" name="laser">
+      <always_on>true</always_on>
+      <visualize>false</visualize>
+      <topic>scan</topic>
+      <update_rate>75.0</update_rate>
+      <plugin name="gazebo_ros_laser_controller" filename="libgazebo_ros_laser.so">
+        <frameName>laser</frameName>
+        <topicName>scan</topicName>
         <gaussianNoise>0.005</gaussianNoise>
-        <alwaysOn>true</alwaysOn>
         <updateRate>75.0</updateRate>
-        <topicName>scan</topicName>
-        <frameName>laser</frameName>
-        <interface:laser name="gazebo_ros_laser_iface" />
-      </controller:gazebo_ros_laser>
-    </sensor:ray>
+      </plugin>
+      <ray>
+        <scan>
+          <horizontal>
+            <samples>181</samples>
+            <resolution>1</resolution>
+            <min_angle>-1.571</min_angle>
+            <max_angle>1.571</max_angle>
+          </horizontal>
+        </scan>
+        <range>
+          <min>0.08</min>
+          <max>10.0</max>
+          <resolution>0.01</resolution>
+        </range>
+      </ray>
+    </sensor>
   </gazebo>
 </robot>
